Commit message: rename arm joints from descriptive names to link numbers

File: cyton_gamma_1500_macros.urdf.xacro (robot description, xacro)
@@ -40,5 +40,5 @@
       </inertial>
     </link>
-    <joint name="${prefix}shoulder_roll_joint" type="revolute">
+    <joint name="${prefix}joint0" type="revolute">
       <parent link="${prefix}base_link" />
       <child link="${prefix}shoulder_roll" />
@@ -67,5 +67,5 @@
       </inertial>
     </link>
-    <joint name="${prefix}shoulder_pitch_joint" type="revolute">
+    <joint name="${prefix}joint1" type="revolute">
       <parent link="${prefix}shoulder_roll" />
       <child link="${prefix}shoulder_pitch" />
@@ -94,5 +94,5 @@
       </inertial>
     </link>
-    <joint name="${prefix}shoulder_yaw_joint" type="revolute">
+    <joint name="${prefix}joint2" type="revolute">
       <parent link="${prefix}shoulder_pitch" />
       <child link="${prefix}shoulder_yaw" />
@@ -121,5 +121,5 @@
       </inertial>
     </link>
-    <joint name="${prefix}elbow_pitch_joint" type="revolute">
+    <joint name="${prefix}joint3" type="revolute">
       <parent link="${prefix}shoulder_yaw" />
       <child link="${prefix}elbow_pitch" />
@@ -148,5 +148,5 @@
       </inertial>
     </link>
-    <joint name="${prefix}elbow_yaw_joint" type="revolute">
+    <joint name="${prefix}joint4" type="revolute">
       <parent link="${prefix}elbow_pitch" />
       <child link="${prefix}elbow_yaw" />
@@ -175,5 +175,5 @@
       </inertial>
     </link>
-    <joint name="${prefix}wrist_pitch_joint" type="revolute">
+    <joint name="${prefix}joint5" type="revolute">
       <parent link="${prefix}elbow_yaw" />
       <child link="${prefix}wrist_pitch" />
@@ -202,5 +202,5 @@
       </inertial>
     </link>
-    <joint name="${prefix}wrist_roll_joint" type="revolute">
+    <joint name="${prefix}joint6" type="revolute">
       <parent link="${prefix}wrist_pitch" />
       <child link="${prefix}wrist_roll" />
@@ -309,5 +309,5 @@
     <plugin name="joint_state_publisher"
             filename="libgazebo_ros_joint_state_publisher.so">
-      <jointName>shoulder_roll_joint, shoulder_pitch_joint, shoulder_yaw_joint, elbow_pitch_joint, elbow_yaw_joint, wrist_pitch_joint, wrist_roll_joint, gripper_joint, gripper_joint2</jointName>
+      <jointName>joint0, joint1, joint2, joint3, joint4, joint5, joint6, gripper_joint, gripper_joint2</jointName>
     </plugin>
   </gazebo>

Commit message: fix collision model

File: cyton_gamma_1500_macros.urdf.xacro (robot description, xacro)
@@ -55,5 +55,5 @@
       </visual>
       <collision>
-        <origin xyz="0.0 0.069 0.0587"/>
+        <origin xyz="0 0 0.0587" rpy="1.5708 0 0"/>
         <geometry>
           <box size="0.09829 0.18143 0.08392"/>
@@ -82,5 +82,5 @@
       </visual>
       <collision>
-        <origin xyz="-0.001 0.064 0.1745"/>
+        <origin xyz="-0.02 -0.001 0.064" rpy="1.5708 0 0"/>
         <geometry>
           <box size="0.0709 0.19363 0.083"/>
@@ -109,5 +109,5 @@
       </visual>
       <collision>
-        <origin xyz="-0.0225 0.039 0.3068"/>
+        <origin xyz="-0.003 0.0225 0.057" rpy="1.5708 0 -1.5708"/>
         <geometry>
           <box size="0.0717 0.1846 0.0756"/>
@@ -136,5 +136,5 @@
       </visual>
       <collision>
-        <origin xyz="0.0346 0.0461 0.4228"/>
+        <origin xyz="-0.017 0.004 0.0461" rpy="1.5708 0 3.1416"/>
         <geometry>
           <box size="0.0549 0.1557 0.076"/>
@@ -163,7 +163,7 @@
       </visual>
       <collision>
-        <origin xyz="0.0172 0.0209 0.516"/>
-        <geometry>
-          <box size="0.0535 0.1160 0.0402"/>
+        <origin xyz="0 0.0172 0.047" rpy="1.5708 0 1.5708" />
+        <geometry>
+          <box size="0.0535 0.1160 0.053"/>
         </geometry>
       </collision>
@@ -190,7 +190,7 @@
       </visual>
       <collision>
-        <origin xyz="0.0257 0.0118 0.5617"/>
-        <geometry>
-          <box size="0.026 0.0435 0.05185"/>
+        <origin xyz="-0.013 0 0.05" rpy="1.5708 0 1.5708" />
+        <geometry>
+          <box size="0.035 0.0435 0.05185"/>
         </geometry>
       </collision>
@@ -217,7 +217,7 @@
       </visual>
       <collision>
-        <origin xyz="-0.0063 -0.0014 0.6102"/>
-        <geometry>
-          <box size="0.0518 0.0723 0.1004"/>
+        <origin xyz="0 0.008 0.05" rpy="3.1416 0 -1.5708"/>
+        <geometry>
+          <box size="0.0518 0.0723 0.06"/>
         </geometry>
       </collision>
@@ -244,5 +244,5 @@
       </visual>
       <collision>
-        <origin xyz="-0.0167 0.0172 0.7254"/>
+        <origin xyz="-0.003 0.01 0.01"/>
         <geometry>
           <box size="0.015 0.0229 0.0475"/>
@@ -272,5 +272,5 @@
       </visual>
       <collision>
-        <origin xyz="0.0132 0.0172 0.7254"/>
+        <origin xyz="0.003 0.01 0.01"/>
         <geometry>
           <box size="0.015 0.0229 0.0475"/>

Commit message: adaptations to URDF model for the simulation to work

File: cyton_gamma_1500_macros.urdf.xacro (robot description, xacro)
@@ -304,7 +304,4 @@
   </xacro:macro>
   <gazebo>
-    <plugin name="gazebo_ros_control" filename="libgazebo_ros_control.so"/>
-  </gazebo>
-  <gazebo>
     <plugin name="joint_state_publisher"
             filename="libgazebo_ros_joint_state_publisher.so">

File: ist_cyton_gamma_1500_macros.urdf.xacro (robot description, xacro)
@@ -1,4 +1,4 @@
 <?xml version="1.0"?>
-<robot xmlns:xacro="http://www.ros.org/wiki/xacro" name="cyton_gamma_1500">
+<robot xmlns:xacro="http://wiki.ros.org/xacro" name="cyton_gamma_1500">
   <!-- math definitions -->
   <xacro:property name="M_PI" value="3.141592653589793" />
@@ -36,5 +36,5 @@
       </collision>
       <inertial>
-        <mass value="100.0"/>
+        <mass value="0.001"/>
         <origin rpy="0 0 0" xyz="0 0 0"/>
         <inertia ixx="1.1027" iyy="1.1027" izz="1.1027"
@@ -63,5 +63,5 @@
       </collision>
       <inertial>
-        <mass value="50.0"/>
+        <mass value="0.001"/>
         <origin rpy="0 0 0" xyz="0 0 0"/>
         <inertia ixx=".1027" iyy=".1027" izz=".1027"
@@ -90,5 +90,5 @@
       </collision>
       <inertial>
-        <mass value="20.0"/>
+        <mass value="0.001"/>
         <origin rpy="0 0 0" xyz="0 0 0"/>
         <inertia ixx=".0827" iyy=".0827" izz=".0827"
@@ -117,5 +117,5 @@
       </collision>
       <inertial>
-        <mass value="10.0"/>
+        <mass value="0.001"/>
         <origin rpy="0 0 0" xyz="0 0 0"/>
         <inertia ixx=".0627" iyy=".0627" izz=".0627"
@@ -144,5 +144,5 @@
       </collision>
       <inertial>
-        <mass value="10.0"/>
+        <mass value="0.001"/>
         <origin rpy="0 0 0" xyz="0 0 0"/>
         <inertia ixx=".0327" iyy=".0327" izz=".0327"
@@ -171,5 +171,5 @@
       </collision>
       <inertial>
-        <mass value="10.0"/>
+        <mass value="0.001"/>
         <origin rpy="0 0 0" xyz="0 0 0"/>
         <inertia ixx=".0227" iyy=".0227" izz=".0227"
@@ -198,5 +198,5 @@
       </collision>
       <inertial>
-        <mass value="10.0"/>
+        <mass value="0.001"/>
         <origin rpy="0 0 0" xyz="0 0 0"/>
         <inertia ixx=".0127" iyy=".0127" izz=".0127"
@@ -225,5 +225,5 @@
       </collision>
       <inertial>
-        <mass value="10.0"/>
+        <mass value="0.001"/>
         <origin rpy="0 0 0" xyz="0 0 0"/>
         <inertia ixx=".0027" iyy=".0027" izz=".0027"
@@ -254,5 +254,5 @@
       </collision>
       <inertial>
-        <mass value="1.0"/>
+        <mass value="0.001"/>
         <origin rpy="0 0 0" xyz="0 0 0"/>
         <inertia ixx=".0027" iyy=".0027" izz=".0027"
@@ -282,8 +282,8 @@
       </collision>
       <inertial>
-        <mass value="1.0"/>
+        <mass value="0.001"/>
         <origin rpy="0 0 0" xyz="0 0 0"/>
         <inertia ixx=".0027" iyy=".0027" izz=".0027"
-                  ixy="0" ixz="0" iyz="0"/>
+                 ixy="0" ixz="0" iyz="0"/>
       </inertial>
     </link>
@@ -308,11 +308,37 @@
   </xacro:macro>
   <gazebo>
-    <plugin name="gazebo_ros_control" filename="libgazebo_ros_control.so"/>
-  </gazebo>
-  <gazebo>
     <plugin name="joint_state_publisher"
             filename="libgazebo_ros_joint_state_publisher.so">
-      <jointName>joint0, joint1, joint2, joint3, joint4, joint5, joint6, gripper_joint, gripper_joint2</jointName>
+      <jointName>left_arm_joint0, left_arm_joint1, left_arm_joint2, left_arm_joint3, left_arm_joint4, left_arm_joint5, left_arm_joint6</jointName>
+      <robotNamespace>/</robotNamespace>
+      <updateRate>50.0</updateRate>
     </plugin>
   </gazebo>
+  <!-- arm transmissions -->
+  <!-- arm transmission macro -->
+  <xacro:macro name="arm_transmission_macro" params="joint_name">
+    <transmission name="${joint_name}_arm_trans">
+      <type>transmission_interface/SimpleTransmission</type>
+      <joint name="${joint_name}">
+        <hardwareInterface>hardware_interface/EffortJointInterface</hardwareInterface>
+      </joint>
+      <actuator name="${joint_name}_actuator">
+        <mechanicalReduction>1</mechanicalReduction>
+      </actuator>
+    </transmission>
+  </xacro:macro>
+  <!-- joint0 -->
+  <xacro:arm_transmission_macro joint_name="left_arm_joint0" />
+  <!-- joint1 -->
+  <xacro:arm_transmission_macro joint_name="left_arm_joint1" />
+  <!-- joint2 -->
+  <xacro:arm_transmission_macro joint_name="left_arm_joint2" />
+  <!-- joint3 -->
+  <xacro:arm_transmission_macro joint_name="left_arm_joint3" />
+  <!-- joint4 -->
+  <xacro:arm_transmission_macro joint_name="left_arm_joint4" />
+  <!-- joint5 -->
+  <xacro:arm_transmission_macro joint_name="left_arm_joint5" />
+  <!-- joint6 -->
+  <xacro:arm_transmission_macro joint_name="left_arm_joint6" />
 </robot>
