Commit message: adjust joint limits on urdf based on bit values tuned in the real arm with dynamixel windows app

File: ist_cyton_gamma_1500_macros.urdf.xacro (robot description, xacro)
@@ -46,5 +46,5 @@
       <child link="${prefix}shoulder_roll" />
       <origin xyz="0 0 0.05315" rpy="0 0 0" />
-      <limit lower="-2.618" upper="2.618" effort="100.0" velocity="1.0" />
+      <limit lower="-2.5509" upper="2.5585" effort="100.0" velocity="1.0" />
       <axis xyz="0 0 1" />
     </joint>
@@ -73,5 +73,5 @@
       <child link="${prefix}shoulder_pitch" />
       <origin xyz="0.0205 0 0.12435" rpy="0 0 0" />
-      <limit lower="-1.8326" upper="1.8326" effort="100.0" velocity="1.0" />
+      <limit lower="-1.707" upper="1.6379" effort="100.0" velocity="1.0" />
       <axis xyz="1 0 0" />
     </joint>
@@ -100,5 +100,5 @@
       <child link="${prefix}shoulder_yaw" />
       <origin xyz="-0.0215 -0.0205 0.1255" rpy="0 0 0" />
-      <limit lower="-1.8326" upper="1.8326" effort="100.0" velocity="1.0" />
+      <limit lower="-1.5459" upper="1.73" effort="100.0" velocity="1.0" />
       <axis xyz="0 -1 0" />
     </joint>
@@ -127,5 +127,5 @@
       <child link="${prefix}elbow_pitch" />
       <origin xyz="0.018 0.0206 0.1158" rpy="0 0 0" />
-      <limit lower="-1.8326" upper="1.8326" effort="100.0" velocity="1.0" />
+      <limit lower="-1.6072" upper="1.6149" effort="100.0" velocity="1.0" />
       <axis xyz="1 0 0" />
     </joint>
@@ -154,5 +154,5 @@
       <child link="${prefix}elbow_yaw" />
       <origin xyz="-0.0171 -0.018 0.09746" rpy="0 0 0" />
-      <limit lower="-1.8326" upper="1.8326" effort="100.0" velocity="1.0" />
+      <limit lower="-1.8757" upper="1.4615" effort="100.0" velocity="1.0" />
       <axis xyz="0 -1 0" />
     </joint>
@@ -181,5 +181,5 @@
       <child link="${prefix}wrist_pitch" />
       <origin xyz="0.02626 0.018 0.0718" rpy="0 0 0" />
-      <limit lower="-1.8326" upper="1.8326" effort="100.0" velocity="1.0" />
+      <limit lower="-1.5766" upper="1.5382" effort="100.0" velocity="1.0" />
       <axis xyz="-1 0 0" />
     </joint>
@@ -208,5 +208,5 @@
       <child link="${prefix}ist_gripper_mount" />
       <origin xyz="-0.026255 0 0.051425" rpy="0 0 0" />
-      <limit lower="-2.61799" upper="2.61799" effort="100.0" velocity="1.0" />
+      <limit lower="-2.5279" upper="2.5355" effort="100.0" velocity="1.0" />
       <axis xyz="0 0 1" />
     </joint>
@@ -235,4 +235,6 @@
       <child link="${prefix}gripper_finger1" />
       <origin xyz="-0.0331 -0.03515 0.098" rpy="${M_PI/2} 0 ${M_PI/2}" />
+      <!-- the following value are for rviz visualization purposes only, real gripper values are : -2.8347, -1.3157 /-->
+      <!-- those values will be normaliezd and republished as sensor_msgs from gripper controller node /-->
       <limit lower="-0.08" upper="0.5" effort="100.0" velocity="1.0" />
       <axis xyz="0 0 1" />
@@ -274,5 +276,4 @@
       </visual>
       <collision>
-        <!--origin xyz="-0.003 0.05 0.015"/-->
         <origin xyz="-0.003 0.05 0.015"/>
         <geometry>

Commit message: fix model angles, matching reality with model, motor turns now in the same direction as described in urdf

File: ist_cyton_gamma_1500_macros.urdf.xacro (robot description, xacro)
@@ -180,5 +180,5 @@
       <parent link="${prefix}elbow_yaw" />
       <child link="${prefix}wrist_pitch" />
-      <origin xyz="0.02626 0.018 0.0718" rpy="0 0 0" />
+      <origin xyz="-0.02626 0.018 0.0718" rpy="0 0 ${M_PI}" />
       <limit lower="-1.5766" upper="1.5382" effort="100.0" velocity="1.0" />
       <axis xyz="-1 0 0" />
@@ -207,5 +207,5 @@
       <parent link="${prefix}wrist_pitch" />
       <child link="${prefix}ist_gripper_mount" />
-      <origin xyz="-0.026255 0 0.051425" rpy="0 0 0" />
+      <origin xyz="-0.026255 0 0.051425" rpy="0 0 ${M_PI/2}" />
       <limit lower="-2.5279" upper="2.5355" effort="100.0" velocity="1.0" />
       <axis xyz="0 0 1" />

Commit message: change virtual end effector link to match with gripper matrix

File: ist_cyton_gamma_1500_macros.urdf.xacro (robot description, xacro)
@@ -288,22 +288,20 @@
       </inertial>
     </link>
-    <xacro:if value="${virtual_ee}"> <!-- virtual end-effector -->
-      <joint name="${prefix}virtual_endeffector_joint" type="fixed">
-        <parent link="${prefix}ist_gripper_mount" />
-        <child link="${prefix}virtual_endeffector" />
-        <origin xyz="-0.002316 0.0079 0.079425" rpy="0 0 0" />
-      </joint>
-      <link name="${prefix}virtual_endeffector">
-        <visual>
-          <origin xyz="0 0 0" rpy="0 0 0" />
-          <geometry>
-            <sphere radius="0.002" />
-          </geometry>
-          <material name="grey">
-            <color rgba="0.7 0.7 0.7 0.8" />
-          </material>
-        </visual>
-      </link>
-    </xacro:if>
+    <joint name="${prefix}virtual_endeffector_joint" type="fixed">
+      <parent link="${prefix}ist_gripper_mount" />
+      <child link="${prefix}virtual_endeffector" />
+      <origin xyz="0.0 0.0 0.17" rpy="0 0 0" />
+    </joint>
+    <link name="${prefix}virtual_endeffector">
+      <visual>
+        <origin xyz="0 0 0" rpy="0 0 0" />
+        <geometry>
+          <sphere radius="0.002" />
+        </geometry>
+        <material name="grey">
+          <color rgba="0.7 0.7 0.7 0.8" />
+        </material>
+      </visual>
+    </link>
   </xacro:macro>
   <gazebo>

Commit message: added collision model for missing links

File: ist_cyton_gamma_1500_macros.urdf.xacro (robot description, xacro)
@@ -243,5 +243,5 @@
         <origin rpy="0.0 0 0" xyz=" 0 -0.045 0"/>
         <geometry>
-          <box size="0.1 0.05 0.1"/>
+          <box size="0.001 0.001 0.001"/>
         </geometry>
       </collision>
@@ -268,5 +268,5 @@
         <origin rpy="0 -0.6 0" xyz="0 0 0"/>
         <geometry>
-          <box size="0.1 0.05 0.1"/>
+          <box size="0.001 0.001 0.001"/>
         </geometry>
       </collision>
@@ -295,5 +295,5 @@
         <origin rpy="0.0 0 0" xyz="0 0 0"/>
         <geometry>
-          <box size="0.1 0.05 0.1"/>
+          <box size="0.001 0.001 0.001"/>
         </geometry>
       </collision>
@@ -323,5 +323,5 @@
         <origin rpy="0 3.142 0" xyz="0 0 0"/>
         <geometry>
-          <box size="0.1 0.05 0.1"/>
+          <box size="0.001 0.001 0.001"/>
         </geometry>
       </collision>
@@ -422,4 +422,5 @@
       <child link="${prefix}two_fingers" />
       <origin xyz="0.06 -0.02 0.0"/>
+ist_cyton_gamma_1500_macros.urdf.xacro
       <axis xyz="0 1 0"/>
       <limit effort="1000.0" lower="0.0" upper="1.68" velocity="0.5"/>

Commit message: organize meshes in folders, fix collision model, delete unnecesary files related with old gripper + other unnecesary files

File: ist_cyton_gamma_1500_macros.urdf.xacro (robot description, xacro)
@@ -28,5 +28,5 @@
         <origin xyz="0 0 0" rpy="0 0 0"/>
         <geometry>
-          <mesh filename="package://cyton_gamma_1500_description/meshes/base.dae"/>
+          <mesh filename="package://cyton_gamma_1500_description/meshes/arm/base.dae"/>
         </geometry>
       </visual>
@@ -55,5 +55,5 @@
         <origin xyz="0 0 0" rpy="0 0 0.384"/>
         <geometry>
-          <mesh filename="package://cyton_gamma_1500_description/meshes/shoulder_roll.dae"/>
+          <mesh filename="package://cyton_gamma_1500_description/meshes/arm/shoulder_roll.dae"/>
         </geometry>
       </visual>
@@ -82,5 +82,5 @@
         <origin xyz="0 0 0" rpy="0 0 0" />
         <geometry>
-          <mesh filename="package://cyton_gamma_1500_description/meshes/shoulder_pitch.dae"/>
+          <mesh filename="package://cyton_gamma_1500_description/meshes/arm/shoulder_pitch.dae"/>
         </geometry>
       </visual>
@@ -109,5 +109,5 @@
         <origin xyz="0 0 0.0" rpy="0 0 -1.5708" />
         <geometry>
-          <mesh filename="package://cyton_gamma_1500_description/meshes/shoulder_yaw.dae"/>
+          <mesh filename="package://cyton_gamma_1500_description/meshes/arm/shoulder_yaw.dae"/>
         </geometry>
       </visual>
@@ -136,5 +136,5 @@
         <origin xyz="0 0 0" rpy="1.5708 0 3.1416" />
         <geometry>
-          <mesh filename="package://cyton_gamma_1500_description/meshes/elbow_pitch.dae"/>
+          <mesh filename="package://cyton_gamma_1500_description/meshes/arm/elbow_pitch.dae"/>
         </geometry>
       </visual>
@@ -163,5 +163,5 @@
         <origin xyz="0 0 0" rpy="0 0 1.5708" />
         <geometry>
-          <mesh filename="package://cyton_gamma_1500_description/meshes/elbow_yaw.dae"/>
+          <mesh filename="package://cyton_gamma_1500_description/meshes/arm/elbow_yaw.dae"/>
         </geometry>
       </visual>
@@ -190,13 +190,7 @@
         <origin xyz="0 0 0" rpy="1.5708 0 1.5708" />
         <geometry>
-          <mesh filename="package://cyton_gamma_1500_description/meshes/wrist_pitch.dae"/>
-        </geometry>
-      </visual>
-      <collision>
-        <origin xyz="-0.02 0 0.05" rpy="1.5708 0 1.5708" />
-        <geometry>
-          <box size="0.085 0.0435 0.05185"/>
-        </geometry>
-      </collision>
+          <mesh filename="package://cyton_gamma_1500_description/meshes/arm/wrist_pitch.dae"/>
+        </geometry>
+      </visual>
       <inertial>
         <mass value="0.001"/>
@@ -217,5 +211,5 @@
         <origin rpy="0.0 0 -1.57" xyz=" -0.013 0.015 0.0359"/>
         <geometry>
-          <mesh filename="package://cyton_gamma_1500_description/meshes/wrist.dae"/>
+          <mesh filename="package://cyton_gamma_1500_description/meshes/arm/wrist.dae"/>
         </geometry>
       </visual>
@@ -223,5 +217,5 @@
         <origin rpy="0.0 0 -1.57" xyz=" -0.013 0.015 0.0359"/>
         <geometry>
-          <box size="0.1 0.05 0.1"/>
+          <box size="0.0001 0.0001 0.0001"/>        <!--0.1 0.05 0.1 -->
         </geometry>
       </collision>
@@ -237,13 +231,7 @@
         <origin rpy="0.0 0 0" xyz=" 0 -0.045 0"/>
         <geometry>
-          <mesh filename="package://cyton_gamma_1500_description/meshes/Motor_+_Base.dae"/>
-        </geometry>
-      </visual>
-      <collision>
-        <origin rpy="0.0 0 0" xyz=" 0 -0.045 0"/>
-        <geometry>
-          <box size="0.1 0.05 0.1"/>
-        </geometry>
-      </collision>
+          <mesh filename="package://cyton_gamma_1500_description/meshes/gripper/Motor_+_Base.dae"/>
+        </geometry>
+      </visual>
       <inertial>
         <mass value="0.001"/>
@@ -262,13 +250,7 @@
         <origin rpy="0 -0.6 0" xyz="0 0 0"/>
         <geometry>
-          <mesh filename="package://cyton_gamma_1500_description/meshes/right_link_front.dae"/>
-        </geometry>
-      </visual>
-      <collision>
-        <origin rpy="0 -0.6 0" xyz="0 0 0"/>
-        <geometry>
-          <box size="0.1 0.05 0.1"/>
-        </geometry>
-      </collision>
+          <mesh filename="package://cyton_gamma_1500_description/meshes/gripper/right_link_front.dae"/>
+        </geometry>
+      </visual>
       <inertial>
         <mass value="0.001"/>
@@ -289,13 +271,7 @@
         <origin rpy="0.0 0 0" xyz="0 0 0"/>
         <geometry>
-          <mesh filename="package://cyton_gamma_1500_description/meshes/right_link_back.dae"/>
-        </geometry>
-      </visual>
-      <collision>
-        <origin rpy="0.0 0 0" xyz="0 0 0"/>
-        <geometry>
-          <box size="0.1 0.05 0.1"/>
-        </geometry>
-      </collision>
+          <mesh filename="package://cyton_gamma_1500_description/meshes/gripper/right_link_back.dae"/>
+        </geometry>
+      </visual>
       <inertial>
         <mass value="0.001"/>
@@ -317,13 +293,7 @@
         <origin rpy="0 3.142 0" xyz="0 0 0"/>
         <geometry>
-          <mesh filename="package://cyton_gamma_1500_description/meshes/left_front_link.dae"/>
-        </geometry>
-      </visual>
-      <collision>
-        <origin rpy="0 3.142 0" xyz="0 0 0"/>
-        <geometry>
-          <box size="0.1 0.05 0.1"/>
-        </geometry>
-      </collision>
+          <mesh filename="package://cyton_gamma_1500_description/meshes/gripper/left_front_link.dae"/>
+        </geometry>
+      </visual>
       <inertial>
         <mass value="0.001"/>
@@ -345,13 +315,7 @@
         <origin rpy="0 3.14 0" xyz="0 0 0"/>
         <geometry>
-          <mesh filename="package://cyton_gamma_1500_description/meshes/left_link_back.dae"/>
-        </geometry>
-      </visual>
-      <collision>
-        <origin rpy="0 3.14 0" xyz="0 0 0"/>
-        <geometry>
-          <box size="0.1 0.05 0.1"/>
-        </geometry>
-      </collision>
+          <mesh filename="package://cyton_gamma_1500_description/meshes/gripper/left_link_back.dae"/>
+        </geometry>
+      </visual>
       <inertial>
         <mass value="0.001"/>
@@ -373,11 +337,11 @@
         <origin rpy="0 0.003 0" xyz="0 0 0"/>
         <geometry>
-          <mesh filename="package://cyton_gamma_1500_description/meshes/one_finger.dae"/>
-        </geometry>
-      </visual>
-      <collision>
-        <origin rpy="0 0.003 0" xyz="0 0 0"/>
-        <geometry>
-          <box size="0.1 0.05 0.1"/>
+          <mesh filename="package://cyton_gamma_1500_description/meshes/gripper/one_finger.dae"/>
+        </geometry>
+      </visual>
+      <collision>
+        <origin rpy="0 -0.05 0" xyz="0.014 -0.001 -0.07"/>
+        <geometry>
+          <box size="0.045 0.025 0.169"/>
         </geometry>
       </collision>
@@ -401,12 +365,11 @@
         <origin rpy="0 0.24 0" xyz="0 0 0"/>
         <geometry>
-          <mesh filename="package://cyton_gamma_1500_description/meshes/two_fingers.dae"/>
-        </geometry>
-        <material name="black"/>
-      </visual>
-      <collision>
-        <origin rpy="0 0.24 0" xyz="0 0 0"/>
-        <geometry>
-          <box size="0.1 0.05 0.1"/>
+          <mesh filename="package://cyton_gamma_1500_description/meshes/gripper/two_fingers.dae"/>
+        </geometry>
+      </visual>
+      <collision>
+        <origin rpy="0 0.1 0" xyz="-0.02 0.024 -0.07"/>
+        <geometry>
+          <box size="0.045 0.07 0.165"/>
         </geometry>
       </collision>
