Commit message: fix harode server merge conflict

File: xacro/ist_cyton_gamma_1500_macros.urdf.xacro (robot description, xacro)
@@ -387,22 +387,20 @@
       <mimic joint="${prefix}gripper_joint" multiplier="-1" offset="0"/>
     </joint>
-    <xacro:if value="${virtual_ee}"> <!-- virtual end-effector -->
-      <joint name="${prefix}virtual_endeffector_joint" type="fixed">
-        <parent link="${prefix}Wrist" />
-        <child link="${prefix}virtual_endeffector" />
-        <origin xyz="-0.002316 0.0079 0.079425" rpy="0 0 0" />
-      </joint>
-      <link name="${prefix}virtual_endeffector">
-        <visual>
-          <origin xyz="0 0 0" rpy="0 0 0" />
-          <geometry>
-            <sphere radius="0.002" />
-          </geometry>
-          <material name="grey">
-            <color rgba="0.7 0.7 0.7 0.8" />
-          </material>
-        </visual>
-      </link>
-    </xacro:if>
+    <joint name="${prefix}virtual_endeffector_joint" type="fixed">
+      <parent link="${prefix}Wrist" />
+      <child link="${prefix}virtual_endeffector" />
+      <origin xyz="-0.002316 0.0079 0.079425" rpy="0 0 0" />
+    </joint>
+    <link name="${prefix}virtual_endeffector">
+      <visual>
+        <origin xyz="0 0 0" rpy="0 0 0" />
+        <geometry>
+          <sphere radius="0.002" />
+        </geometry>
+        <material name="grey">
+          <color rgba="0.7 0.7 0.7 0.8" />
+        </material>
+      </visual>
+    </link>
   </xacro:macro>
   <gazebo>
@@ -442,5 +440,7 @@
   <!-- joint6 -->
   <xacro:arm_transmission_macro joint_name="left_arm_joint6" />
-  <!-- gripper joint -->
+  <!-- gripper joint 1 -->
   <xacro:arm_transmission_macro joint_name="left_arm_gripper_joint" />
+  <!-- gripper joint 2 (fake mirror joint)-->
+  <xacro:arm_transmission_macro joint_name="left_arm_gripper_joint2" />
 </robot>

Commit message: fix end effector pose, delete left_arm_gripper_joint2 from model

File: xacro/ist_cyton_gamma_1500_macros.urdf.xacro (robot description, xacro)
@@ -388,7 +388,7 @@
     </joint>
     <joint name="${prefix}virtual_endeffector_joint" type="fixed">
-      <parent link="${prefix}Wrist" />
+      <parent link="${prefix}Motor_+_Base" />
       <child link="${prefix}virtual_endeffector" />
-      <origin xyz="-0.002316 0.0079 0.079425" rpy="0 0 0" />
+      <origin xyz="-0.002316 0.0079 -0.12" rpy="0 0 0" />
     </joint>
     <link name="${prefix}virtual_endeffector">
@@ -404,5 +404,5 @@
     </link>
   </xacro:macro>
-  <gazebo>
+  <!--<gazebo>
     <plugin name="joint_state_publisher"
             filename="libgazebo_ros_joint_state_publisher.so">
@@ -412,5 +412,5 @@
       <updateRate>50.0</updateRate>
     </plugin>
-  </gazebo>
+  </gazebo>-->
   <!-- arm transmissions -->
   <!-- arm transmission macro (needed for Gazebo simulator -->
@@ -442,5 +442,3 @@
   <!-- gripper joint 1 -->
   <xacro:arm_transmission_macro joint_name="left_arm_gripper_joint" />
-  <!-- gripper joint 2 (fake mirror joint)-->
-  <xacro:arm_transmission_macro joint_name="left_arm_gripper_joint2" />
 </robot>

Commit message: change in axis of rotation for gripper to match real robot

File: xacro/ist_cyton_gamma_1500_macros.urdf.xacro (robot description, xacro)
@@ -263,5 +263,5 @@
       <origin xyz="0 0 0 "/>
       <limit effort="1000.0" lower="0.0" upper="1.68" velocity="0.5"/>
-      <axis xyz="0 1 0" />
+      <axis xyz="0 -1 0" />
     </joint>
     <link name="${prefix}right_link_back">

Commit message: fix gripper urdf model, gripper finger going in oposite direction

File: xacro/ist_cyton_gamma_1500_macros.urdf.xacro (robot description, xacro)
@@ -263,5 +263,5 @@
       <origin xyz="0 0 0 "/>
       <limit effort="1000.0" lower="0.0" upper="1.68" velocity="0.5"/>
-      <axis xyz="0 -1 0" />
+      <axis xyz="0 1 0" />
     </joint>
     <link name="${prefix}right_link_back">

Commit message: fix wrong rotation direction of joint 6 mbot arm (last joint)

File: xacro/ist_cyton_gamma_1500_macros.urdf.xacro (robot description, xacro)
@@ -203,5 +203,5 @@
       <origin rpy="0 3.14 0" xyz="-0.026255 0.0 0.115"/>
       <limit lower="-2.5279" upper="2.5355" effort="100.0" velocity="1.0" />
-      <axis xyz="0 0 1" />
+      <axis xyz="0 0 -1" />
     </joint>
     <link name="${prefix}Wrist">

Commit message: fix gripper joint limits on urdf model

File: xacro/ist_cyton_gamma_1500_macros.urdf.xacro (robot description, xacro)
@@ -262,5 +262,5 @@
       <child link="${prefix}right_link_front" />
       <origin xyz="0 0 0 "/>
-      <limit effort="1000.0" lower="0.0" upper="1.68" velocity="0.5"/>
+      <limit effort="1000.0" lower="-1.5" upper="-0.1" velocity="0.5"/>
       <axis xyz="0 1 0" />
     </joint>

Commit message: delete unnecesary stuff from arm urdf

File: xacro/ist_cyton_gamma_1500_macros.urdf.xacro (robot description, xacro)
@@ -3,23 +3,5 @@
   <!-- math definitions -->
   <xacro:property name="M_PI" value="3.141592653589793" />
-  <xacro:macro name="base_footprint" params="prefix">
-    <link name="${prefix}base_footprint">
-      <visual>
-        <origin xyz="0 0 0" rpy="0 0 0"/>
-        <geometry>
-          <sphere radius="0.001" />
-        </geometry>
-        <material name="white">
-          <color rgba="1 1 1 1"/>
-        </material>
-      </visual>
-    </link>
-    <joint name="base_joint" type="fixed">
-      <parent link="${prefix}base_footprint" />
-      <child link="${prefix}base_link" />
-      <origin xyz="0.0 0.0 0.0" rpy="0 0 0" />
-    </joint>
-  </xacro:macro>
-  <xacro:macro name="cyton_gamma_1500" params="prefix virtual_ee">
+  <xacro:macro name="cyton_gamma_1500" params="prefix">
     <link name="${prefix}base_link">
       <visual>

Commit message: generalize mimic joints to accept angular offset and tune for real arm offset

File: xacro/ist_cyton_gamma_1500_macros.urdf.xacro (robot description, xacro)
@@ -3,4 +3,9 @@
   <!-- math definitions -->
   <xacro:property name="M_PI" value="3.141592653589793" />
+  <!-- gripper joint limits -->
+  <xacro:property name="gripper_lower_limit" value="-1.5" />
+  <xacro:property name="gripper_upper_limit" value="-0.1" />
+  <xacro:property name="gripper_angular_offset" value="1.75" />
+  <!-- arm macro definition -->
   <xacro:macro name="cyton_gamma_1500" params="prefix">
     <link name="${prefix}base_link">
@@ -243,6 +248,6 @@
       <parent link="${prefix}Motor_+_Base" />
       <child link="${prefix}right_link_front" />
-      <origin xyz="0 0 0 "/>
-      <limit effort="1000.0" lower="-1.5" upper="-0.1" velocity="0.5"/>
+      <origin xyz="0 0 0" rpy="0 ${gripper_angular_offset} 0" />
+      <limit effort="1000.0" lower="${gripper_lower_limit}" upper="${gripper_upper_limit}" velocity="0.5"/>
       <axis xyz="0 1 0" />
     </joint>
@@ -264,7 +269,7 @@
       <parent link="${prefix}Motor_+_Base" />
       <child link="${prefix}right_link_back" />
-      <origin xyz="0.025 -0.0085 0.015 "/>
-      <axis xyz="0 1 0"/>
-      <limit effort="1000.0" lower="0.0" upper="1.68" velocity="0.5"/>
+      <origin xyz="0.025 -0.0085 0.015" rpy="0 ${gripper_angular_offset} 0" />
+      <axis xyz="0 1 0" />
+      <limit effort="1000.0" lower="${gripper_lower_limit}" upper="${gripper_upper_limit}" velocity="0.5"/>
       <mimic joint="${prefix}gripper_joint" multiplier="1" offset="0"/>
     </joint>
@@ -286,7 +291,7 @@
       <parent link="${prefix}Motor_+_Base" />
       <child link="${prefix}left_link_front" />
-      <origin xyz="-0.022 -0.001 0"/>
-      <axis xyz="0 1 0"/>
-      <limit effort="1000.0" lower="0.0" upper="1.68" velocity="0.5"/>
+      <origin xyz="-0.022 -0.001 0" rpy="0 -${gripper_angular_offset} 0" />
+      <axis xyz="0 1 0" />
+      <limit effort="1000.0" lower="${gripper_lower_limit}" upper="${gripper_upper_limit}" velocity="0.5"/>
       <mimic joint="${prefix}gripper_joint" multiplier="-1" offset="0"/>
     </joint>
@@ -308,7 +313,7 @@
       <parent link="${prefix}Motor_+_Base" />
       <child link="${prefix}left_link_back" />
-      <origin xyz="-0.0469 -0.014 0.0155"/>
-      <axis xyz="0 1 0"/>
-      <limit effort="1000.0" lower="0.0" upper="1.68" velocity="0.5"/>
+      <origin xyz="-0.0469 -0.014 0.0155" rpy="0 -${gripper_angular_offset} 0" />
+      <axis xyz="0 1 0" />
+      <limit effort="1000.0" lower="${gripper_lower_limit}" upper="${gripper_upper_limit}" velocity="0.5"/>
       <mimic joint="${prefix}gripper_joint" multiplier="-1" offset="0"/>
     </joint>
@@ -336,7 +341,7 @@
       <parent link="${prefix}left_link_back" />
       <child link="${prefix}one_finger" />
-      <origin xyz="-0.06 0.008 0.0"/>
-      <axis xyz="0 1 0"/>
-      <limit effort="1000.0" lower="0.0" upper="1.68" velocity="0.5"/>
+      <origin xyz="-0.06 0.008 0.0" rpy="0 ${gripper_angular_offset} 0" />
+      <axis xyz="0 1 0" />
+      <limit effort="1000.0" lower="${gripper_lower_limit}" upper="${gripper_upper_limit}" velocity="0.5"/>
       <mimic joint="${prefix}motor_base_to_left_link_front" multiplier="-1" offset="0"/>
     </joint>
@@ -364,7 +369,7 @@
       <parent link="${prefix}right_link_back" />
       <child link="${prefix}two_fingers" />
-      <origin xyz="0.06 -0.02 0.0"/>
-      <axis xyz="0 1 0"/>
-      <limit effort="1000.0" lower="0.0" upper="1.68" velocity="0.5"/>
+      <origin xyz="0.06 -0.02 0.0" rpy="0 -${gripper_angular_offset} 0" />
+      <axis xyz="0 1 0" />
+      <limit effort="1000.0" lower="${gripper_lower_limit}" upper="${gripper_upper_limit}" velocity="0.5"/>
       <mimic joint="${prefix}gripper_joint" multiplier="-1" offset="0"/>
     </joint>

Commit message: make joint mimic the gripper instead of the other mimic to fix gripper not being able to actuate in gazebo and not publishing joint states in rviz

File: xacro/ist_cyton_gamma_1500_macros.urdf.xacro (robot description, xacro)
@@ -344,5 +344,5 @@
       <axis xyz="0 1 0" />
       <limit effort="1000.0" lower="${gripper_lower_limit}" upper="${gripper_upper_limit}" velocity="0.5"/>
-      <mimic joint="${prefix}motor_base_to_left_link_front" multiplier="-1" offset="0"/>
+      <mimic joint="${prefix}gripper_joint" multiplier="1" offset="0"/>
     </joint>
     <link name="${prefix}two_fingers">

Commit message: [gripper sim] solve problem of mbot gripper not able to actuate by using gazebo mimic joint plugin

File: xacro/ist_cyton_gamma_1500_macros.urdf.xacro (robot description, xacro)
@@ -293,5 +293,5 @@
       <origin xyz="-0.022 -0.001 0" rpy="0 -${gripper_angular_offset} 0" />
       <axis xyz="0 1 0" />
-      <limit effort="1000.0" lower="${gripper_lower_limit}" upper="${gripper_upper_limit}" velocity="0.5"/>
+      <limit effort="1000.0" lower="${-gripper_upper_limit}" upper="${-gripper_lower_limit}" velocity="0.5"/>
       <mimic joint="${prefix}gripper_joint" multiplier="-1" offset="0"/>
     </joint>
@@ -315,5 +315,5 @@
       <origin xyz="-0.0469 -0.014 0.0155" rpy="0 -${gripper_angular_offset} 0" />
       <axis xyz="0 1 0" />
-      <limit effort="1000.0" lower="${gripper_lower_limit}" upper="${gripper_upper_limit}" velocity="0.5"/>
+      <limit effort="1000.0" lower="${-gripper_upper_limit}" upper="${-gripper_lower_limit}" velocity="0.5"/>
       <mimic joint="${prefix}gripper_joint" multiplier="-1" offset="0"/>
     </joint>
@@ -371,5 +371,5 @@
       <origin xyz="0.06 -0.02 0.0" rpy="0 -${gripper_angular_offset} 0" />
       <axis xyz="0 1 0" />
-      <limit effort="1000.0" lower="${gripper_lower_limit}" upper="${gripper_upper_limit}" velocity="0.5"/>
+      <limit effort="1000.0" lower="${-gripper_upper_limit}" upper="${-gripper_lower_limit}" velocity="0.5"/>
       <mimic joint="${prefix}gripper_joint" multiplier="-1" offset="0"/>
     </joint>
@@ -391,5 +391,24 @@
     </link>
   </xacro:macro>
-  <!--<gazebo>
+  <!-- plugin to support mimic joints in gazebo -->
+  <xacro:macro name="mimic_joints_macro" params="joint_to_be_mimiced mimic_joint multiplier">
+    <gazebo>
+      <plugin name="${mimic_joint}_mimic_plugin" filename="libroboticsgroup_gazebo_mimic_joint_plugin.so" >
+          <joint>left_arm_${joint_to_be_mimiced}</joint>
+          <mimicJoint>left_arm_${mimic_joint}</mimicJoint>
+          <multiplier>${multiplier}</multiplier>
+          <offset>0.0</offset>
+      </plugin>
+    </gazebo>
+  </xacro:macro>
+  <!-- left side of gripper -->
+  <xacro:mimic_joints_macro joint_to_be_mimiced="gripper_joint" mimic_joint="motor_base_to_left_link_front" multiplier="-1.0" />
+  <xacro:mimic_joints_macro joint_to_be_mimiced="gripper_joint" mimic_joint="motor_base_to_left_link_back" multiplier="-1.0" />
+  <xacro:mimic_joints_macro joint_to_be_mimiced="gripper_joint" mimic_joint="left_link_back_to_one_finger" multiplier="1.0" />
+  <!-- right side of gripper -->
+  <!-- right_link_front is actuated by gripper joint, therefore no need for mimic plugin -->
+  <xacro:mimic_joints_macro joint_to_be_mimiced="gripper_joint" mimic_joint="motor_base_to_right_link_back" multiplier="1.0" />
+  <xacro:mimic_joints_macro joint_to_be_mimiced="gripper_joint" mimic_joint="right_link_back_to_two_fingers" multiplier="-1.0" />
+  <!--<gazebo> ROS control publishes joint states currently, so no need for gazebo to do it
     <plugin name="joint_state_publisher"
             filename="libgazebo_ros_joint_state_publisher.so">
@@ -400,6 +419,5 @@
     </plugin>
   </gazebo>-->
-  <!-- arm transmissions -->
-  <!-- arm transmission macro (needed for Gazebo simulator -->
+  <!-- arm transmission macro (needed to actuate joints in gazebo simulator via ROS control) -->
   <xacro:macro name="arm_transmission_macro" params="joint_name">
     <transmission name="${joint_name}_arm_trans">

Commit message: replace harcoded small mass with variable to set all at once

File: xacro/ist_cyton_gamma_1500_macros.urdf.xacro (robot description, xacro)
@@ -7,4 +7,6 @@
   <xacro:property name="gripper_upper_limit" value="-0.1" />
   <xacro:property name="gripper_angular_offset" value="1.75" />
+  <!-- small mass that can be set to all links -->
+  <xacro:property name="small_mass" value="0.00001" />
   <!-- arm macro definition -->
   <xacro:macro name="cyton_gamma_1500" params="prefix">
@@ -23,5 +25,5 @@
       </collision>
       <inertial>
-        <mass value="0.001"/>
+        <mass value="${small_mass}" />
         <origin rpy="0 0 0" xyz="0 0 0"/>
         <inertia ixx="1.1027" iyy="1.1027" izz="1.1027"
@@ -50,5 +52,5 @@
       </collision>
       <inertial>
-        <mass value="0.001"/>
+        <mass value="${small_mass}" />
         <origin rpy="0 0 0" xyz="0 0 0"/>
         <inertia ixx=".1027" iyy=".1027" izz=".1027"
@@ -77,5 +79,5 @@
       </collision>
       <inertial>
-        <mass value="0.001"/>
+        <mass value="${small_mass}" />
         <origin rpy="0 0 0" xyz="0 0 0"/>
         <inertia ixx=".0827" iyy=".0827" izz=".0827"
@@ -104,5 +106,5 @@
       </collision>
       <inertial>
-        <mass value="0.001"/>
+        <mass value="${small_mass}" />
         <origin rpy="0 0 0" xyz="0 0 0"/>
         <inertia ixx=".0627" iyy=".0627" izz=".0627"
@@ -131,5 +133,5 @@
       </collision>
       <inertial>
-        <mass value="0.001"/>
+        <mass value="${small_mass}" />
         <origin rpy="0 0 0" xyz="0 0 0"/>
         <inertia ixx=".0327" iyy=".0327" izz=".0327"
@@ -158,5 +160,5 @@
       </collision>
       <inertial>
-        <mass value="0.001"/>
+        <mass value="${small_mass}" />
         <origin rpy="0 0 0" xyz="0 0 0"/>
         <inertia ixx=".0227" iyy=".0227" izz=".0227"
@@ -179,5 +181,5 @@
       </visual>
       <inertial>
-        <mass value="0.001"/>
+        <mass value="${small_mass}" />
         <origin rpy="0 0 0" xyz="0 0 0"/>
         <inertia ixx=".0127" iyy=".0127" izz=".0127"
@@ -206,5 +208,5 @@
       </collision>
       <inertial>
-        <mass value="0.001"/>
+        <mass value="${small_mass}" />
         <origin rpy="0 0 0" xyz="0 0 0"/>
         <inertia ixx=".0027" iyy=".0027" izz=".0027"
@@ -220,5 +222,5 @@
       </visual>
       <inertial>
-        <mass value="0.001"/>
+        <mass value="${small_mass}" />
         <origin rpy="0 0 0" xyz="0 0 0"/>
         <inertia ixx=".0027" iyy=".0027" izz=".0027"
@@ -239,5 +241,5 @@
       </visual>
       <inertial>
-        <mass value="0.001"/>
+        <mass value="${small_mass}" />
         <origin rpy="0 0 0" xyz="0 0 0"/>
         <inertia ixx=".0027" iyy=".0027" izz=".0027"
@@ -260,5 +262,5 @@
       </visual>
       <inertial>
-        <mass value="0.001"/>
+        <mass value="${small_mass}" />
         <origin rpy="0 0 0" xyz="0 0 0"/>
         <inertia ixx=".0027" iyy=".0027" izz=".0027"
@@ -282,5 +284,5 @@
       </visual>
       <inertial>
-        <mass value="0.001"/>
+        <mass value="${small_mass}" />
         <origin rpy="0 0 0" xyz="0 0 0"/>
         <inertia ixx=".0027" iyy=".0027" izz=".0027"
@@ -304,5 +306,5 @@
       </visual>
       <inertial>
-        <mass value="0.001"/>
+        <mass value="${small_mass}" />
         <origin rpy="0 0 0" xyz="0 0 0"/>
         <inertia ixx=".0027" iyy=".0027" izz=".0027"
@@ -332,5 +334,5 @@
       </collision>
       <inertial>
-        <mass value="0.001"/>
+        <mass value="${small_mass}" />
         <origin rpy="0 0 0" xyz="0 0 0"/>
         <inertia ixx=".0027" iyy=".0027" izz=".0027"
@@ -360,5 +362,5 @@
       </collision>
       <inertial>
-        <mass value="0.001"/>
+        <mass value="${small_mass}" />
         <origin rpy="0 0 0" xyz="0 0 0"/>
         <inertia ixx=".0027" iyy=".0027" izz=".0027"

Commit message: fix bug where gripper is shaking

File: xacro/ist_cyton_gamma_1500_macros.urdf.xacro (robot description, xacro)
@@ -8,5 +8,7 @@
   <xacro:property name="gripper_angular_offset" value="1.75" />
   <!-- small mass that can be set to all links -->
-  <xacro:property name="small_mass" value="0.00001" />
+  <xacro:property name="small_mass" value="0.0001" />
+  <!-- we dont know yet the moment of inertia of the robot! -->
+  <xacro:property name="small_inertial_value" value="0.01" />
   <!-- arm macro definition -->
   <xacro:macro name="cyton_gamma_1500" params="prefix">
@@ -180,9 +182,15 @@
         </geometry>
       </visual>
-      <inertial>
+      <!--inertial>
         <mass value="${small_mass}" />
         <origin rpy="0 0 0" xyz="0 0 0"/>
         <inertia ixx=".0127" iyy=".0127" izz=".0127"
                   ixy="0" ixz="0" iyz="0"/>
+      </inertial-->
+      <inertial>
+        <mass value="${small_mass}"/>
+        <origin rpy="0 0 0" xyz="0 0 0"/>
+        <inertia ixx="${small_inertial_value}" ixy="0" ixz="0"
+                iyy="${small_inertial_value}" iyz="0" izz="${small_inertial_value}"/>
       </inertial>
     </link>
@@ -208,8 +216,8 @@
       </collision>
       <inertial>
-        <mass value="${small_mass}" />
-        <origin rpy="0 0 0" xyz="0 0 0"/>
-        <inertia ixx=".0027" iyy=".0027" izz=".0027"
-                  ixy="0" ixz="0" iyz="0"/>
+        <mass value="${small_mass}"/>
+        <origin rpy="0 0 0" xyz="0 0 0"/>
+        <inertia ixx="${small_inertial_value}" ixy="0" ixz="0"
+                iyy="${small_inertial_value}" iyz="0" izz="${small_inertial_value}"/>
       </inertial>
     </link>
@@ -222,8 +230,8 @@
       </visual>
       <inertial>
-        <mass value="${small_mass}" />
-        <origin rpy="0 0 0" xyz="0 0 0"/>
-        <inertia ixx=".0027" iyy=".0027" izz=".0027"
-                  ixy="0" ixz="0" iyz="0"/>
+        <mass value="${small_mass}"/>
+        <origin rpy="0 0 0" xyz="0 0 0"/>
+        <inertia ixx="${small_inertial_value}" ixy="0" ixz="0"
+                iyy="${small_inertial_value}" iyz="0" izz="${small_inertial_value}"/>
       </inertial>
     </link>
@@ -241,8 +249,8 @@
       </visual>
       <inertial>
-        <mass value="${small_mass}" />
-        <origin rpy="0 0 0" xyz="0 0 0"/>
-        <inertia ixx=".0027" iyy=".0027" izz=".0027"
-                  ixy="0" ixz="0" iyz="0"/>
+        <mass value="${small_mass}"/>
+        <origin rpy="0 0 0" xyz="0 0 0"/>
+        <inertia ixx="${small_inertial_value}" ixy="0" ixz="0"
+                iyy="${small_inertial_value}" iyz="0" izz="${small_inertial_value}"/>
       </inertial>
     </link>
@@ -262,8 +270,8 @@
       </visual>
       <inertial>
-        <mass value="${small_mass}" />
-        <origin rpy="0 0 0" xyz="0 0 0"/>
-        <inertia ixx=".0027" iyy=".0027" izz=".0027"
-                 ixy="0" ixz="0" iyz="0"/>
+        <mass value="${small_mass}"/>
+        <origin rpy="0 0 0" xyz="0 0 0"/>
+        <inertia ixx="${small_inertial_value}" ixy="0" ixz="0"
+                iyy="${small_inertial_value}" iyz="0" izz="${small_inertial_value}"/>
       </inertial>
     </link>
@@ -284,8 +292,8 @@
       </visual>
       <inertial>
-        <mass value="${small_mass}" />
-        <origin rpy="0 0 0" xyz="0 0 0"/>
-        <inertia ixx=".0027" iyy=".0027" izz=".0027"
-                  ixy="0" ixz="0" iyz="0"/>
+        <mass value="${small_mass}"/>
+        <origin rpy="0 0 0" xyz="0 0 0"/>
+        <inertia ixx="${small_inertial_value}" ixy="0" ixz="0"
+                iyy="${small_inertial_value}" iyz="0" izz="${small_inertial_value}"/>
       </inertial>
     </link>
@@ -306,8 +314,8 @@
       </visual>
       <inertial>
-        <mass value="${small_mass}" />
-        <origin rpy="0 0 0" xyz="0 0 0"/>
-        <inertia ixx=".0027" iyy=".0027" izz=".0027"
-                 ixy="0" ixz="0" iyz="0"/>
+        <mass value="${small_mass}"/>
+        <origin rpy="0 0 0" xyz="0 0 0"/>
+        <inertia ixx="${small_inertial_value}" ixy="0" ixz="0"
+                iyy="${small_inertial_value}" iyz="0" izz="${small_inertial_value}"/>
       </inertial>
     </link>
@@ -334,8 +342,8 @@
       </collision>
       <inertial>
-        <mass value="${small_mass}" />
-        <origin rpy="0 0 0" xyz="0 0 0"/>
-        <inertia ixx=".0027" iyy=".0027" izz=".0027"
-                  ixy="0" ixz="0" iyz="0"/>
+        <mass value="${small_mass}"/>
+        <origin rpy="0 0 0" xyz="0 0 0"/>
+        <inertia ixx="${small_inertial_value}" ixy="0" ixz="0"
+                iyy="${small_inertial_value}" iyz="0" izz="${small_inertial_value}"/>
       </inertial>
     </link>
@@ -362,8 +370,8 @@
       </collision>
       <inertial>
-        <mass value="${small_mass}" />
-        <origin rpy="0 0 0" xyz="0 0 0"/>
-        <inertia ixx=".0027" iyy=".0027" izz=".0027"
-                  ixy="0" ixz="0" iyz="0"/>
+        <mass value="${small_mass}"/>
+        <origin rpy="0 0 0" xyz="0 0 0"/>
+        <inertia ixx="${small_inertial_value}" ixy="0" ixz="0"
+                iyy="${small_inertial_value}" iyz="0" izz="${small_inertial_value}"/>
       </inertial>
     </link>
