Commit message: The robots xacro file was updated with a new camera attached on the robots arm.

File: xacro/ist_cyton_gamma_1500_macros.urdf.xacro (robot description, xacro)
@@ -3,4 +3,6 @@
   <!-- math definitions -->
   <xacro:property name="M_PI" value="3.141592653589793" />
+  <!-- Camera -->
+  <xacro:property name="camera_size_link" value="0.008" />
   <!-- gripper joint limits -->
   <xacro:property name="gripper_lower_limit" value="-1.5" />
@@ -492,4 +494,102 @@
       </visual>
     </link>
+    <!-- Camera -->
+    <!-- Camera: Colour : Base_Camera_link -->
+    <gazebo reference="${prefix}base_camera_link">
+      <material>Gazebo/FlatBlack</material>
+    </gazebo>
+    <!-- Camera: Colour : Camera_link -->
+    <gazebo reference="${prefix}camera_link">
+      <material>Gazebo/RedTransparent</material>
+    </gazebo>
+    <!-- Camera: Joint : Wrist to Base_Camera -->
+    <joint name="${prefix}joint_base_camera" type="fixed">
+      <origin xyz="0 0 0.02" rpy="0 0 0"/>
+      <parent link="${prefix}Wrist" />
+      <child link="${prefix}base_camera_link" />
+    </joint>
+    <!-- Camera: Base Camera Link -->
+    <link name="${prefix}base_camera_link">
+      <collision>
+        <origin xyz="0 0.03 0" rpy="0 0 0"/>
+        <geometry>
+          <box size="0.01 0.05 0.01"/>
+        </geometry>
+      </collision>
+      <visual>
+        <origin xyz="0 0.03 0" rpy="0 0 0"/>
+        <geometry>
+          <box size="0.01 0.05 0.01"/>
+        </geometry>
+      </visual>
+      <inertial>
+        <mass value="0.01" />
+        <origin xyz="0 0.03 0" rpy="0 0 0"/>
+        <inertia ixx="1.666666e-07" ixy="0.0" ixz="0.0" iyy="1.666666e-07" iyz="0.0" izz="1.666666e-07"/>
+      </inertial>
+    </link>
+    <!-- Camera: Joint : Base_Camera to Camera -->
+    <joint name="{prefix}camera_link" type="fixed">
+      <origin xyz="0 0.05 -0.005" rpy="-1.7 1.7 0"/>
+      <parent link="${prefix}base_camera_link"/>
+      <child link="${prefix}camera_link"/>
+    </joint>
+    <!-- Camera -->
+    <link name="${prefix}camera_link">
+      <collision>
+        <origin xyz="0 0 0" rpy="0 0 0"/>
+        <geometry>
+          <box size="${camera_size_link} ${camera_size_link} ${camera_size_link}"/>
+        </geometry>
+      </collision>
+      <visual>
+        <origin xyz="0 0 0" rpy="0 0 0"/>
+        <geometry>
+          <box size="${camera_size_link} ${camera_size_link} ${camera_size_link}"/>
+        </geometry>
+      </visual>
+      <inertial>
+        <mass value="1e-5" />
+        <origin xyz="0 0 0" rpy="0 0 0"/>
+        <inertia ixx="1e-6" ixy="0" ixz="0" iyy="1e-6" iyz="0" izz="1e-6" />
+      </inertial>
+    </link>
+    <!-- Camera: plugin -->
+    <gazebo reference="${prefix}camera_link">
+      <sensor type="camera" name="camera_grasping">
+        <update_rate>30.0</update_rate>
+        <camera name="head">
+          <horizontal_fov>1.3962634</horizontal_fov>
+          <image>
+            <width>800</width>
+            <height>800</height>
+            <format>R8G8B8</format>
+          </image>
+          <clip>
+            <near>0.02</near>
+            <far>300</far>
+          </clip>
+          <noise>
+            <type>gaussian</type>
+            <mean>0.0</mean>
+            <stddev>0.007</stddev>
+          </noise>
+        </camera>
+        <plugin name="camera_controller" filename="libgazebo_ros_camera.so">
+          <alwaysOn>true</alwaysOn>
+          <updateRate>0.0</updateRate>
+          <cameraName>camera_grasping</cameraName>
+          <imageTopicName>image_grasping</imageTopicName>
+          <cameraInfoTopicName>camera_info</cameraInfoTopicName>
+          <frameName>camera_link</frameName>
+          <hackBaseline>0.07</hackBaseline>
+          <distortionK1>0.0</distortionK1>
+          <distortionK2>0.0</distortionK2>
+          <distortionK3>0.0</distortionK3>
+          <distortionT1>0.0</distortionT1>
+          <distortionT2>0.0</distortionT2>
+        </plugin>
+      </sensor>
+     </gazebo>
     <!-- to attach objects when grasping -->
     <gazebo>

Commit message: Removed some unnecessary comments and changed the signature of the new camera topic.

File: xacro/ist_cyton_gamma_1500_macros.urdf.xacro (robot description, xacro)
@@ -28,10 +28,4 @@
         </geometry>
       </collision>
-      <!--inertial>
-        <mass value="${small_mass}" />
-        <origin rpy="0 0 0" xyz="0 0 0"/>
-        <inertia ixx="1.1027" iyy="1.1027" izz="1.1027"
-                 ixy="0" ixz="0" iyz="0"/>
-      </inertial-->
       <inertial>
         <mass value="0.1"/>
@@ -60,10 +54,4 @@
         </geometry>
       </collision>
-      <!--inertial>
-        <mass value="${small_mass}" />
-        <origin rpy="0 0 0" xyz="0 0 0"/>
-        <inertia ixx=".1027" iyy=".1027" izz=".1027"
-                 ixy="0" ixz="0" iyz="0"/>
-      </inertial-->
       <inertial>
         <mass value="0.1"/>
@@ -92,10 +80,4 @@
         </geometry>
       </collision>
-      <!--inertial>
-        <mass value="${small_mass}" />
-        <origin rpy="0 0 0" xyz="0 0 0"/>
-        <inertia ixx=".0827" iyy=".0827" izz=".0827"
-                 ixy="0" ixz="0" iyz="0"/>
-      </inertial-->
       <inertial>
         <mass value="0.1"/>
@@ -124,10 +106,4 @@
         </geometry>
       </collision>
-      <!--inertial>
-        <mass value="${small_mass}" />
-        <origin rpy="0 0 0" xyz="0 0 0"/>
-        <inertia ixx=".0627" iyy=".0627" izz=".0627"
-                 ixy="0" ixz="0" iyz="0"/>
-      </inertial-->
       <inertial>
         <mass value="0.1"/>
@@ -156,10 +132,4 @@
         </geometry>
       </collision>
-      <!--inertial>
-        <mass value="${small_mass}" />
-        <origin rpy="0 0 0" xyz="0 0 0"/>
-        <inertia ixx=".0327" iyy=".0327" izz=".0327"
-                 ixy="0" ixz="0" iyz="0"/>
-      </inertial-->
       <inertial>
         <mass value="0.1"/>
@@ -188,10 +158,4 @@
         </geometry>
       </collision>
-      <!--inertial>
-        <mass value="${small_mass}" />
-        <origin rpy="0 0 0" xyz="0 0 0"/>
-        <inertia ixx=".0227" iyy=".0227" izz=".0227"
-                 ixy="0" ixz="0" iyz="0"/>
-      </inertial-->
       <inertial>
         <mass value="0.1"/>
@@ -219,10 +183,4 @@
         <inertia ixx="9.0833297e-05" ixy="0.0" ixz="0.0" iyy="1.4999994e-05" iyz="0.0" izz="9.0833297e-05"/>
       </inertial>
-      <!--inertial>
-        <mass value="0.0001"/>
-        <origin xyz="0 0 0" rpy="1.5708 0 1.5708" />
-        <inertia ixx="0.01" ixy="0" ixz="0"
-                 iyy="0.01" iyz="0" izz="0.01"/>
-      </inertial-->
     </link>
     <joint name="${prefix}joint6" type="revolute">
@@ -246,27 +204,34 @@
         </geometry>
       </collision>
-      <!--inertial>
+      <inertial>
+        <mass value="0.1"/>
+        <origin xyz="0 0 -0.04"/>
+        <inertia ixx="0.00055768311026" ixy="0.0" ixz="0.0" iyy="0.00050976646276" iyz="0.0" izz="0.0001154166205"/>
+      </inertial>
+    </link>
+    <link name="${prefix}Motor_+_Base">
+      <visual>
+        <origin rpy="0.0 0 0" xyz=" 0 -0.045 0"/>
+        <geometry>
+          <mesh filename="package://cyton_gamma_1500_description/meshes/gripper/Motor_+_Base.dae"/>
+        </geometry>
+      </visual>
+      <inertial>
         <mass value="${small_mass}"/>
         <origin rpy="0 0 0" xyz="0 0 0"/>
         <inertia ixx="${small_inertial_value}" ixy="0" ixz="0"
                 iyy="${small_inertial_value}" iyz="0" izz="${small_inertial_value}"/>
-      </inertial-->
-      <inertial>
-        <mass value="0.1"/>
-        <origin xyz="0 0 -0.04"/>
-        <inertia ixx="0.00055768311026" ixy="0.0" ixz="0.0" iyy="0.00050976646276" iyz="0.0" izz="0.0001154166205"/>
-        <!--inertia ixx="0.001372499451" ixy="0.0" ixz="0.0" iyy="0.001372499451" iyz="0.0" izz="0.00112499955"/-->
-        <!--inertia ixx="0.001884999246" ixy="0.0" ixz="0.0" iyy="0.001884999246" iyz="0.0" izz="0.00112499955"/-->
-        <!--mass value="0.0001"/>
-        <origin rpy="0 0 0" xyz="0 0 0"/>
-        <inertia ixx="0.01" ixy="0" ixz="0"
-                 iyy="0.01" iyz="0" izz="0.01"/-->
-      </inertial>
-    </link>
-    <link name="${prefix}Motor_+_Base">
-      <visual>
-        <origin rpy="0.0 0 0" xyz=" 0 -0.045 0"/>
-        <geometry>
-          <mesh filename="package://cyton_gamma_1500_description/meshes/gripper/Motor_+_Base.dae"/>
+      </inertial>
+    </link>
+    <joint name="${prefix}wrist_to_motor_+_base" type="fixed">
+      <parent link="${prefix}Wrist" />
+      <child link="${prefix}Motor_+_Base" />
+      <origin xyz="0 0.022 0"/>
+    </joint>
+    <link name="${prefix}right_link_front">
+      <visual>
+        <origin rpy="0 -0.6 0" xyz="0 0 0"/>
+        <geometry>
+          <mesh filename="package://cyton_gamma_1500_description/meshes/gripper/right_link_front.dae"/>
         </geometry>
       </visual>
@@ -277,28 +242,4 @@
                 iyy="${small_inertial_value}" iyz="0" izz="${small_inertial_value}"/>
       </inertial>
-    </link>
-    <joint name="${prefix}wrist_to_motor_+_base" type="fixed">
-      <parent link="${prefix}Wrist" />
-      <child link="${prefix}Motor_+_Base" />
-      <origin xyz="0 0.022 0"/>
-    </joint>
-    <link name="${prefix}right_link_front">
-      <visual>
-        <origin rpy="0 -0.6 0" xyz="0 0 0"/>
-        <geometry>
-          <mesh filename="package://cyton_gamma_1500_description/meshes/gripper/right_link_front.dae"/>
-        </geometry>
-      </visual>
-      <inertial>
-        <mass value="${small_mass}"/>
-        <origin rpy="0 0 0" xyz="0 0 0"/>
-        <inertia ixx="${small_inertial_value}" ixy="0" ixz="0"
-                iyy="${small_inertial_value}" iyz="0" izz="${small_inertial_value}"/>
-      </inertial>
-      <!--inertial>
-         <mass value="0.01"/>
-         <origin xyz="0.05 0 0"/>
-         <inertia ixx="5.24370614418e-07" ixy="0.0" ixz="0.0" iyy="5.16033748003e-06" iyz="0.0" izz="4.77857097524e-06"/>
-       </inertial-->
     </link>
     <joint name="${prefix}gripper_joint" type="revolute">
@@ -328,9 +269,4 @@
                 iyy="${small_inertial_value}" iyz="0" izz="${small_inertial_value}"/>
       </inertial>
-      <!--inertial>
-        <mass value="0.01"/>
-        <origin xyz="0.04 0 0"/>
-        <inertia ixx="5.24370614418e-07" ixy="0.0" ixz="0.0" iyy="5.16033748003e-06" iyz="0.0" izz="4.77857097524e-06"/>
-      </inertial-->
     </link>
     <joint name="${prefix}motor_base_to_right_link_back" type="revolute">
@@ -355,9 +291,4 @@
                 iyy="${small_inertial_value}" iyz="0" izz="${small_inertial_value}"/>
       </inertial>
-      <!--inertial>
-         <mass value="0.01"/>
-         <origin xyz="-0.05 0 0"/>
-         <inertia ixx="5.24370614418e-07" ixy="0.0" ixz="0.0" iyy="5.16033748003e-06" iyz="0.0" izz="4.77857097524e-06"/>
-       </inertial-->
     </link>
     <joint name="${prefix}motor_base_to_left_link_front" type="revolute">
@@ -388,9 +319,4 @@
                 iyy="${small_inertial_value}" iyz="0" izz="${small_inertial_value}"/>
       </inertial>
-      <!--inertial>
-        <mass value="0.01"/>
-        <origin xyz="-0.04 0 0"/>
-        <inertia ixx="5.24370614418e-07" ixy="0.0" ixz="0.0" iyy="5.16033748003e-06" iyz="0.0" izz="4.77857097524e-06"/>
-      </inertial-->
     </link>
     <joint name="${prefix}motor_base_to_left_link_back" type="revolute">
@@ -415,10 +341,4 @@
         </geometry>
       </collision>
-      <!--inertial>
-        <mass value="0.0001"/>
-        <origin rpy="0 0 0" xyz="0 0 0"/>
-        <inertia ixx="0.01" ixy="0" ixz="0"
-                iyy="0.01" iyz="0" izz="0.01"/>
-      </inertial-->
       <inertial>
         <mass value="0.1"/>
@@ -448,10 +368,4 @@
         </geometry>
       </collision>
-      <!--inertial>
-        <mass value="0.0001"/>
-        <origin rpy="0 0 0" xyz="0 0 0"/>
-        <inertia ixx="0.01" ixy="0" ixz="0"
-                iyy="0.01" iyz="0" izz="0.01"/>
-      </inertial-->
       <inertial>
         <mass value="0.1"/>
@@ -579,6 +493,6 @@
           <alwaysOn>true</alwaysOn>
           <updateRate>0.0</updateRate>
-          <cameraName>camera_grasping</cameraName>
-          <imageTopicName>image_grasping</imageTopicName>
+          <cameraName>gripper_camera</cameraName>
+          <imageTopicName>image_raw</imageTopicName>
           <cameraInfoTopicName>camera_info</cameraInfoTopicName>
           <frameName>camera_link</frameName>
