Commit message: going back to old big inertia and add plugins to attach object and put camera on the gripper

File: xacro/ist_cyton_gamma_1500_macros.urdf.xacro (robot description, xacro)
@@ -10,7 +10,7 @@
   <xacro:property name="gripper_angular_offset" value="1.75" />
   <!-- small mass that can be set to all links -->
-  <xacro:property name="small_mass" value="0.01" />
+  <xacro:property name="small_mass" value="0.0001" />
   <!-- we dont know yet the moment of inertia of the robot! -->
-  <xacro:property name="small_inertial_value" value="0.00001" />
+  <xacro:property name="small_inertial_value" value="0.01" />
   <!-- arm macro definition -->
   <xacro:macro name="cyton_gamma_1500" params="prefix">
@@ -29,7 +29,8 @@
       </collision>
       <inertial>
-        <mass value="0.1"/>
-        <origin xyz="0 0.0115 0.047"/>
-        <inertia ixx="0.00033470819945" ixy="0.0" ixz="0.0" iyy="0.00027126655816" iyz="0.0" izz="0.00045870814985"/>
+        <mass value="${small_mass}" />
+        <origin rpy="0 0 0" xyz="0 0 0"/>
+        <inertia ixx="1.1027" iyy="1.1027" izz="1.1027"
+                 ixy="0" ixz="0" iyz="0"/>
       </inertial>
     </link>
@@ -55,7 +56,8 @@
       </collision>
       <inertial>
-        <mass value="0.1"/>
-        <origin xyz="0 0 0.0587" rpy="1.5708 0 0"/>
-        <inertia ixx="0.000332994960969" ixy="0.0" ixz="0.0" iyy="0.000139195698488" iyz="0.0" izz="0.000354814599741"/>
+        <mass value="${small_mass}" />
+        <origin rpy="0 0 0" xyz="0 0 0"/>
+        <inertia ixx=".1027" iyy=".1027" izz=".1027"
+                 ixy="0" ixz="0" iyz="0"/>
       </inertial>
     </link>
@@ -81,7 +83,8 @@
       </collision>
       <inertial>
-        <mass value="0.1"/>
-        <origin xyz="-0.02 -0.001 0.064" rpy="1.5708 0 0"/>
-        <inertia ixx="0.000369846326228" ixy="0.0" ixz="0.0" iyy="9.92983769473e-05" iyz="0.0" izz="0.000354328082435"/>
+        <mass value="${small_mass}" />
+        <origin rpy="0 0 0" xyz="0 0 0"/>
+        <inertia ixx=".0827" iyy=".0827" izz=".0827"
+                 ixy="0" ixz="0" iyz="0"/>
       </inertial>
     </link>
@@ -107,7 +110,8 @@
       </collision>
       <inertial>
-        <mass value="0.1"/>
-        <origin xyz="-0.003 0.0225 0.057" rpy="1.5708 0 -1.5708"/>
-        <inertia ixx="0.000331604200692" ixy="0.0" ixz="0.0" iyy="9.04687138125e-05" iyz="0.0" izz="0.000326816952606"/>
+        <mass value="${small_mass}" />
+        <origin rpy="0 0 0" xyz="0 0 0"/>
+        <inertia ixx=".0627" iyy=".0627" izz=".0627"
+                 ixy="0" ixz="0" iyz="0"/>
       </inertial>
     </link>
@@ -133,7 +137,8 @@
       </collision>
       <inertial>
-        <mass value="0.1"/>
-        <origin xyz="-0.017 0.004 0.0461" rpy="1.5708 0 3.1416"/>
-        <inertia ixx="0.000250153983272" ixy="0.0" ixz="0.0" iyy="7.32500540333e-05" iyz="0.0" izz="0.000227137409145"/>
+        <mass value="${small_mass}" />
+        <origin rpy="0 0 0" xyz="0 0 0"/>
+        <inertia ixx=".0327" iyy=".0327" izz=".0327"
+                 ixy="0" ixz="0" iyz="0"/>
       </inertial>
     </link>
@@ -159,7 +164,8 @@
       </collision>
       <inertial>
-        <mass value="0.1"/>
-        <origin xyz="0 0.0172 0.047" rpy="1.5708 0 1.5708"/>
-        <inertia ixx="0.00013554161245" ixy="0.0" ixz="0.0" iyy="4.72603977625e-05" iyz="0.0" izz="0.000135985362272"/>
+        <mass value="${small_mass}" />
+        <origin rpy="0 0 0" xyz="0 0 0"/>
+        <inertia ixx=".0227" iyy=".0227" izz=".0227"
+                 ixy="0" ixz="0" iyz="0"/>
       </inertial>
     </link>
@@ -178,8 +184,15 @@
         </geometry>
       </visual>
-      <inertial>
-        <mass value="0.1"/>
-        <origin xyz="-0.03 0 0.03" rpy="1.5708 0 1.5708" />
-        <inertia ixx="9.0833297e-05" ixy="0.0" ixz="0.0" iyy="1.4999994e-05" iyz="0.0" izz="9.0833297e-05"/>
+      <!--inertial>
+        <mass value="${small_mass}" />
+        <origin rpy="0 0 0" xyz="0 0 0"/>
+        <inertia ixx=".0127" iyy=".0127" izz=".0127"
+                  ixy="0" ixz="0" iyz="0"/>
+      </inertial-->
+      <inertial>
+        <mass value="${small_mass}"/>
+        <origin rpy="0 0 0" xyz="0 0 0"/>
+        <inertia ixx="${small_inertial_value}" ixy="0" ixz="0"
+                iyy="${small_inertial_value}" iyz="0" izz="${small_inertial_value}"/>
       </inertial>
     </link>
@@ -199,13 +212,14 @@
       </visual>
       <collision>
-        <origin rpy="0.0 0 -1.57" xyz="-0.013 0 0.0359"/>
-        <geometry>
-          <box size="0.07 0.07 0.1"/>        <!--0.1 0.05 0.1 -->
-        </geometry>
-      </collision>
-      <inertial>
-        <mass value="0.1"/>
-        <origin xyz="0 0 -0.04"/>
-        <inertia ixx="0.00055768311026" ixy="0.0" ixz="0.0" iyy="0.00050976646276" iyz="0.0" izz="0.0001154166205"/>
+        <origin rpy="0.0 0 -1.57" xyz=" -0.013 0.015 0.0359"/>
+        <geometry>
+          <box size="0.0001 0.0001 0.0001"/>        <!--0.1 0.05 0.1 -->
+        </geometry>
+      </collision>
+      <inertial>
+        <mass value="${small_mass}"/>
+        <origin rpy="0 0 0" xyz="0 0 0"/>
+        <inertia ixx="${small_inertial_value}" ixy="0" ixz="0"
+                iyy="${small_inertial_value}" iyz="0" izz="${small_inertial_value}"/>
       </inertial>
     </link>
@@ -257,10 +271,4 @@
         </geometry>
       </visual>
-      <collision>
-        <origin rpy="0 -1.6 0" xyz="0.03 0 0"/>
-        <geometry>
-          <box size="0.02 0.02 0.07"/>
-        </geometry>
-      </collision>
       <inertial>
         <mass value="${small_mass}"/>
@@ -307,10 +315,4 @@
         </geometry>
       </visual>
-      <collision>
-         <origin rpy="0 1.6 0" xyz="-0.03 0 0"/>
-         <geometry>
-          <box size="0.02 0.02 0.07"/>
-        </geometry>
-      </collision>
       <inertial>
         <mass value="${small_mass}"/>
@@ -336,13 +338,14 @@
       </visual>
       <collision>
-        <origin rpy="0 0 0" xyz="0.014 -0.001 -0.07"/>
-        <geometry>
-          <box size="0.045 0.07 0.169"/>
-        </geometry>
-      </collision>
-      <inertial>
-        <mass value="0.1"/>
-        <origin xyz="0.01 0 -0.07" rpy="0 0 0"/>
-        <inertia ixx="0.00027884155513" ixy="0.0" ixz="0.0" iyy="0.00025488323138" iyz="0.0" izz="5.770831025e-05"/>
+        <origin rpy="0 -0.05 0" xyz="0.014 -0.001 -0.07"/>
+        <geometry>
+          <box size="0.045 0.025 0.169"/>
+        </geometry>
+      </collision>
+      <inertial>
+        <mass value="${small_mass}"/>
+        <origin rpy="0 0 0" xyz="0 0 0"/>
+        <inertia ixx="${small_inertial_value}" ixy="0" ixz="0"
+                iyy="${small_inertial_value}" iyz="0" izz="${small_inertial_value}"/>
       </inertial>
     </link>
@@ -363,5 +366,5 @@
       </visual>
       <collision>
-        <origin rpy="0 0 0" xyz="-0.02 0.024 -0.07"/>
+        <origin rpy="0 0.1 0" xyz="-0.02 0.024 -0.07"/>
         <geometry>
           <box size="0.045 0.07 0.165"/>
@@ -369,17 +372,18 @@
       </collision>
       <inertial>
-        <mass value="0.1"/>
-        <origin xyz="-0.02 0.03 -0.07" rpy="0 0 0"/>
-        <inertia ixx="0.00026770822625" ixy="0.0" ixz="0.0" iyy="0.0002437499025" iyz="0.0" izz="5.770831025e-05"/>
+        <mass value="${small_mass}"/>
+        <origin rpy="0 0 0" xyz="0 0 0"/>
+        <inertia ixx="${small_inertial_value}" ixy="0" ixz="0"
+                iyy="${small_inertial_value}" iyz="0" izz="${small_inertial_value}"/>
       </inertial>
     </link>
     <gazebo reference="${prefix}one_finger">
-      <mu1 value="1"/>
-      <mu2 value="1"/>
+      <mu1 value="50.0"/>
+      <mu2 value="50.0"/> <!-- enable gripper finger friction-->
       <material>Gazebo/DepthMapVS</material>
     </gazebo>
     <gazebo reference="${prefix}two_fingers">
-      <mu1 value="1"/>
-      <mu2 value="1"/>
+      <mu1 value="50.0"/>
+      <mu2 value="50.0"/> <!-- enable gripper fingers friction-->
       <material>Gazebo/DepthMapVS</material>
     </gazebo>
@@ -505,24 +509,35 @@
         </plugin>
       </sensor>
-     </gazebo>
-    <!-- to attach objects when grasping -->
+    </gazebo>
+   <!-- to attach objects when grasping -->
     <gazebo>
-        <plugin name="gazebo_grasp_fix" filename="libgazebo_grasp_fix.so">
-            <arm>
-                <arm_name>${prefix}</arm_name>
-                <palm_link>${prefix}Wrist</palm_link>
-                <gripper_link>${prefix}one_finger</gripper_link>
-                <gripper_link>${prefix}two_fingers</gripper_link>
-            </arm>
-            <forces_angle_tolerance>100</forces_angle_tolerance>
-            <update_rate>4</update_rate>
-            <grip_count_threshold>4</grip_count_threshold>
-            <max_grip_count>8</max_grip_count>
-            <release_tolerance>0.005</release_tolerance>
-            <disable_collisions_on_attach>false</disable_collisions_on_attach>
-            <contact_topic>__default_topic__</contact_topic>
-        </plugin>
+      <plugin name="gazebo_grasp_fix" filename="libgazebo_grasp_fix.so">
+        <arm>
+        <arm_name>${prefix}</arm_name>
+          <palm_link>${prefix}Wrist</palm_link>
+          <gripper_link>${prefix}one_finger</gripper_link>
+          <gripper_link>${prefix}two_fingers</gripper_link>
+        </arm>
+        <forces_angle_tolerance>100</forces_angle_tolerance>
+        <update_rate>4</update_rate>
+        <grip_count_threshold>4</grip_count_threshold>
+        <max_grip_count>8</max_grip_count>
+        <release_tolerance>0.005</release_tolerance>
+        <disable_collisions_on_attach>false</disable_collisions_on_attach>
+        <contact_topic>__default_topic__</contact_topic>
+      </plugin>
     </gazebo>
   </xacro:macro> <!-- end of mbot arm macro -->
+  <!-- plugin to support mimic joints in gazebo -->
+  <xacro:macro name="mimic_joints_macro" params="joint_to_be_mimiced mimic_joint multiplier">
+    <gazebo>
+      <plugin name="${mimic_joint}_mimic_plugin" filename="libroboticsgroup_gazebo_mimic_joint_plugin.so" >
+        <joint>left_arm_${joint_to_be_mimiced}</joint>
+        <mimicJoint>left_arm_${mimic_joint}</mimicJoint>
+        <multiplier>${multiplier}</multiplier>
+        <offset>0.0</offset>
+      </plugin>
+    </gazebo>
+  </xacro:macro>
   <!-- plugin to support mimic joints in gazebo -->
   <xacro:macro name="mimic_joints_macro" params="joint_to_be_mimiced mimic_joint multiplier">
@@ -581,13 +596,3 @@
   <!-- gripper joint 1 -->
   <xacro:arm_transmission_macro joint_name="left_arm_gripper_joint" />
-  <!-- arm transmission macro based on effort for gripper -->
-    <!--transmission name="left_arm_gripper_joint_arm_trans">
-      <type>transmission_interface/SimpleTransmission</type>
-      <joint name="left_arm_gripper_joint">
-        <hardwareInterface>hardware_interface/EffortJointInterface</hardwareInterface>
-      </joint>
-      <actuator name="left_arm_gripper_joint_actuator">
-        <mechanicalReduction>1</mechanicalReduction>
-      </actuator>
-    </transmission-->
 </robot>

Commit message: change parent of virtual endeffector from Motor_+_Base to Wrist, plus calibrating transform

File: xacro/ist_cyton_gamma_1500_macros.urdf.xacro (robot description, xacro)
@@ -397,7 +397,7 @@
     </joint>
     <joint name="${prefix}virtual_endeffector_joint" type="fixed">
-      <parent link="${prefix}Motor_+_Base" />
+      <parent link="${prefix}Wrist" />
       <child link="${prefix}virtual_endeffector" />
-      <origin xyz="-0.002316 0.0079 -0.12" rpy="0 0 0" />
+      <origin xyz="-0.012 0.018 -0.130" rpy="0 0 0" /> <!-- set this value also in mbot pregrasp planning gripper matrix -->
     </joint>
     <link name="${prefix}virtual_endeffector">

Commit message: add collision box to wrist link to prevent objects to slip while grasping

File: xacro/ist_cyton_gamma_1500_macros.urdf.xacro (robot description, xacro)
@@ -211,8 +211,14 @@
         </geometry>
       </visual>
-      <collision>
+      <!--collision>
         <origin rpy="0.0 0 -1.57" xyz=" -0.013 0.015 0.0359"/>
         <geometry>
-          <box size="0.0001 0.0001 0.0001"/>        <!--0.1 0.05 0.1 -->
+          <box size="0.0001 0.0001 0.0001"/>
+        </geometry>
+      </collision-->
+      <collision>
+        <origin rpy="0.0 0 -1.57" xyz="-0.013 0 0.0359"/>
+        <geometry>
+          <box size="0.06 0.09 0.1"/>
         </geometry>
       </collision>

Commit message: remove repeated plugin

File: xacro/ist_cyton_gamma_1500_macros.urdf.xacro (robot description, xacro)
@@ -535,15 +535,4 @@
     </gazebo>
   </xacro:macro> <!-- end of mbot arm macro -->
-  <!-- plugin to support mimic joints in gazebo -->
-  <xacro:macro name="mimic_joints_macro" params="joint_to_be_mimiced mimic_joint multiplier">
-    <gazebo>
-      <plugin name="${mimic_joint}_mimic_plugin" filename="libroboticsgroup_gazebo_mimic_joint_plugin.so" >
-        <joint>left_arm_${joint_to_be_mimiced}</joint>
-        <mimicJoint>left_arm_${mimic_joint}</mimicJoint>
-        <multiplier>${multiplier}</multiplier>
-        <offset>0.0</offset>
-      </plugin>
-    </gazebo>
-  </xacro:macro>
   <!-- plugin to support mimic joints in gazebo -->
   <xacro:macro name="mimic_joints_macro" params="joint_to_be_mimiced mimic_joint multiplier">
