Commit message: New inertia for the arm. It prevents the undesired behaviour when switching controller from position to velocity.

File: xacro/ist_cyton_gamma_1500_macros.urdf.xacro (robot description, xacro)
@@ -28,9 +28,14 @@
         </geometry>
       </collision>
-      <inertial>
+      <!--inertial>
         <mass value="${small_mass}" />
         <origin rpy="0 0 0" xyz="0 0 0"/>
         <inertia ixx="1.1027" iyy="1.1027" izz="1.1027"
                  ixy="0" ixz="0" iyz="0"/>
+      </inertial-->
+      <inertial>
+        <mass value="1.4"/>
+        <origin xyz="0 0 0"/>
+        <inertia ixx="0.2248838665" ixy="0.0" ixz="0.0" iyy="0.224890078997" iyz="0.0" izz="0.000661645568675"/>
       </inertial>
     </link>
@@ -55,9 +60,14 @@
         </geometry>
       </collision>
-      <inertial>
+      <!--inertial>
         <mass value="${small_mass}" />
         <origin rpy="0 0 0" xyz="0 0 0"/>
         <inertia ixx=".1027" iyy=".1027" izz=".1027"
                  ixy="0" ixz="0" iyz="0"/>
+      </inertial-->
+      <inertial>
+        <mass value="40"/> <!-- This needs to be calculated different because it is a different kind of torque -->
+        <origin xyz="0 0 0"/>
+        <inertia ixx="0.133197984387" ixy="0.0" ixz="0.0" iyy="0.141925839896" iyz="0.0" izz="0.0556782793953"/>
       </inertial>
     </link>
@@ -82,9 +92,14 @@
         </geometry>
       </collision>
-      <inertial>
+      <!--inertial>
         <mass value="${small_mass}" />
         <origin rpy="0 0 0" xyz="0 0 0"/>
         <inertia ixx=".0827" iyy=".0827" izz=".0827"
                  ixy="0" ixz="0" iyz="0"/>
+      </inertial-->
+      <inertial>
+        <mass value="1"/>
+        <origin xyz="0 0 0"/>
+        <inertia ixx="0.103266402435" ixy="0.0" ixz="0.0" iyy="0.103270839933" iyz="0.0" izz="0.000472603977625"/>
       </inertial>
     </link>
@@ -109,9 +124,14 @@
         </geometry>
       </collision>
-      <inertial>
-        <mass value="${small_mass}" />
+      <!--inertial>
+        <mass value="${small_mass}"/>
         <origin rpy="0 0 0" xyz="0 0 0"/>
         <inertia ixx=".0627" iyy=".0627" izz=".0627"
                  ixy="0" ixz="0" iyz="0"/>
+      </inertial-->
+      <inertial>
+        <mass value="0.8"/>
+        <origin xyz="0 0 0"/>
+        <inertia ixx="0.0564055701044" ixy="0.0" ixz="0.0" iyy="0.056409120103" iyz="0.0" izz="0.0003780831821"/>
       </inertial>
     </link>
@@ -136,9 +156,14 @@
         </geometry>
       </collision>
-      <inertial>
+      <!--inertial>
         <mass value="${small_mass}" />
         <origin rpy="0 0 0" xyz="0 0 0"/>
         <inertia ixx=".0327" iyy=".0327" izz=".0327"
                  ixy="0" ixz="0" iyz="0"/>
+      </inertial-->
+      <inertial>
+        <mass value="0.6"/>
+        <origin xyz="0 0 0"/>
+        <inertia ixx="0.0270562236775" ixy="0.0" ixz="0.0" iyy="0.0270588861764" iyz="0.0" izz="0.000283562386575"/>
       </inertial>
     </link>
@@ -163,9 +188,14 @@
         </geometry>
       </collision>
-      <inertial>
+      <!--inertial>
         <mass value="${small_mass}" />
         <origin rpy="0 0 0" xyz="0 0 0"/>
         <inertia ixx=".0227" iyy=".0227" izz=".0227"
                  ixy="0" ixz="0" iyz="0"/>
+      </inertial-->
+      <inertial>
+        <mass value="0.45"/>
+        <origin xyz="0 0 0"/>
+        <inertia ixx="0.0126334824466" ixy="0.0" ixz="0.0" iyy="0.0126354793208" iyz="0.0" izz="0.000212671789931"/>
       </inertial>
     </link>
@@ -190,9 +220,14 @@
                   ixy="0" ixz="0" iyz="0"/>
       </inertial-->
-      <inertial>
-        <mass value="${small_mass}"/>
-        <origin rpy="0 0 0" xyz="0 0 0"/>
-        <inertia ixx="${small_inertial_value}" ixy="0" ixz="0"
-                iyy="${small_inertial_value}" iyz="0" izz="${small_inertial_value}"/>
+      <!--inertial>
+        <mass value="${small_mass}"/>
+        <origin rpy="0 0 0" xyz="0 0 0"/>
+        <inertia ixx="${small_inertial_value}" ixy="0" ixz="0"
+                iyy="${small_inertial_value}" iyz="0" izz="${small_inertial_value}"/>
+      </inertial-->
+      <inertial>
+        <mass value="0.3"/>
+        <origin xyz="0 0 0"/>
+        <inertia ixx="0.00540632283747" ixy="0.0" ixz="0.0" iyy="0.00540765408694" iyz="0.0" izz="0.000141781193287"/>
       </inertial>
     </link>
@@ -211,10 +246,4 @@
         </geometry>
       </visual>
-      <!--collision>
-        <origin rpy="0.0 0 -1.57" xyz=" -0.013 0.015 0.0359"/>
-        <geometry>
-          <box size="0.0001 0.0001 0.0001"/>
-        </geometry>
-      </collision-->
       <collision>
         <origin rpy="0.0 0 -1.57" xyz="-0.013 0 0.0359"/>
@@ -223,9 +252,14 @@
         </geometry>
       </collision>
-      <inertial>
-        <mass value="${small_mass}"/>
-        <origin rpy="0 0 0" xyz="0 0 0"/>
-        <inertia ixx="${small_inertial_value}" ixy="0" ixz="0"
-                iyy="${small_inertial_value}" iyz="0" izz="${small_inertial_value}"/>
+      <!--inertial>
+        <mass value="${small_mass}"/>
+        <origin rpy="0 0 0" xyz="0 0 0"/>
+        <inertia ixx="${small_inertial_value}" ixy="0" ixz="0"
+                iyy="${small_inertial_value}" iyz="0" izz="${small_inertial_value}"/>
+      </inertial-->
+      <inertial>
+        <mass value="0.5"/>
+        <origin xyz="0 0 0"/>
+        <inertia ixx="0.00067770806225" ixy="0.0" ixz="0.0" iyy="0.000679926811362" iyz="0.0" izz="0.000236301988812"/>
       </inertial>
     </link>
@@ -237,9 +271,14 @@
         </geometry>
       </visual>
-      <inertial>
-        <mass value="${small_mass}"/>
-        <origin rpy="0 0 0" xyz="0 0 0"/>
-        <inertia ixx="${small_inertial_value}" ixy="0" ixz="0"
-                iyy="${small_inertial_value}" iyz="0" izz="${small_inertial_value}"/>
+      <!--inertial>
+        <mass value="${small_mass}"/>
+        <origin rpy="0 0 0" xyz="0 0 0"/>
+        <inertia ixx="${small_inertial_value}" ixy="0" ixz="0"
+                iyy="${small_inertial_value}" iyz="0" izz="${small_inertial_value}"/>
+      </inertial-->
+      <inertial>
+        <mass value="0.08"/>
+        <origin rpy="0 0 0" xyz="0 0 0"/>
+        <inertia ixx="0.00010843328996" ixy="0.0" ixz="0.0" iyy="0.000108788289818" iyz="0.0" izz="3.780831821e-05"/>
       </inertial>
     </link>
@@ -256,9 +295,14 @@
         </geometry>
       </visual>
-      <inertial>
-        <mass value="${small_mass}"/>
-        <origin rpy="0 0 0" xyz="0 0 0"/>
-        <inertia ixx="${small_inertial_value}" ixy="0" ixz="0"
-                iyy="${small_inertial_value}" iyz="0" izz="${small_inertial_value}"/>
+      <!--inertial>
+        <mass value="${small_mass}"/>
+        <origin rpy="0 0 0" xyz="0 0 0"/>
+        <inertia ixx="${small_inertial_value}" ixy="0" ixz="0"
+                iyy="${small_inertial_value}" iyz="0" izz="${small_inertial_value}"/>
+      </inertial-->
+      <inertial>
+        <mass value="0.03"/>
+        <origin rpy="0 0 0" xyz="0 0 0"/>
+        <inertia ixx="4.4999982e-06" ixy="0.0" ixz="0.0" iyy="4.4999982e-06" iyz="0.0" izz="4.4999982e-06"/>
       </inertial>
     </link>
@@ -277,9 +321,14 @@
         </geometry>
       </visual>
-      <inertial>
-        <mass value="${small_mass}"/>
-        <origin rpy="0 0 0" xyz="0 0 0"/>
-        <inertia ixx="${small_inertial_value}" ixy="0" ixz="0"
-                iyy="${small_inertial_value}" iyz="0" izz="${small_inertial_value}"/>
+      <!--inertial>
+        <mass value="${small_mass}"/>
+        <origin rpy="0 0 0" xyz="0 0 0"/>
+        <inertia ixx="${small_inertial_value}" ixy="0" ixz="0"
+                iyy="${small_inertial_value}" iyz="0" izz="${small_inertial_value}"/>
+      </inertial-->
+      <inertial>
+        <mass value="0.03"/>
+        <origin rpy="0 0 0" xyz="0 0 0"/>
+        <inertia ixx="4.4999982e-06" ixy="0.0" ixz="0.0" iyy="4.4999982e-06" iyz="0.0" izz="4.4999982e-06"/>
       </inertial>
     </link>
@@ -299,9 +348,14 @@
         </geometry>
       </visual>
-      <inertial>
-        <mass value="${small_mass}"/>
-        <origin rpy="0 0 0" xyz="0 0 0"/>
-        <inertia ixx="${small_inertial_value}" ixy="0" ixz="0"
-                iyy="${small_inertial_value}" iyz="0" izz="${small_inertial_value}"/>
+      <!--inertial>
+        <mass value="${small_mass}"/>
+        <origin rpy="0 0 0" xyz="0 0 0"/>
+        <inertia ixx="${small_inertial_value}" ixy="0" ixz="0"
+                iyy="${small_inertial_value}" iyz="0" izz="${small_inertial_value}"/>
+      </inertial-->
+      <inertial>
+        <mass value="0.03"/>
+        <origin rpy="0 0 0" xyz="0 0 0"/>
+        <inertia ixx="4.4999982e-06" ixy="0.0" ixz="0.0" iyy="4.4999982e-06" iyz="0.0" izz="4.4999982e-06"/>
       </inertial>
     </link>
@@ -321,9 +375,14 @@
         </geometry>
       </visual>
-      <inertial>
-        <mass value="${small_mass}"/>
-        <origin rpy="0 0 0" xyz="0 0 0"/>
-        <inertia ixx="${small_inertial_value}" ixy="0" ixz="0"
-                iyy="${small_inertial_value}" iyz="0" izz="${small_inertial_value}"/>
+      <!--inertial>
+        <mass value="${small_mass}"/>
+        <origin rpy="0 0 0" xyz="0 0 0"/>
+        <inertia ixx="${small_inertial_value}" ixy="0" ixz="0"
+                iyy="${small_inertial_value}" iyz="0" izz="${small_inertial_value}"/>
+      </inertial-->
+      <inertial>
+        <mass value="0.03"/>
+        <origin rpy="0 0 0" xyz="0 0 0"/>
+        <inertia ixx="4.4999982e-06" ixy="0.0" ixz="0.0" iyy="4.4999982e-06" iyz="0.0" izz="4.4999982e-06"/>
       </inertial>
     </link>
@@ -349,9 +408,14 @@
         </geometry>
       </collision>
-      <inertial>
-        <mass value="${small_mass}"/>
-        <origin rpy="0 0 0" xyz="0 0 0"/>
-        <inertia ixx="${small_inertial_value}" ixy="0" ixz="0"
-                iyy="${small_inertial_value}" iyz="0" izz="${small_inertial_value}"/>
+      <!--inertial>
+        <mass value="${small_mass}"/>
+        <origin rpy="0 0 0" xyz="0 0 0"/>
+        <inertia ixx="${small_inertial_value}" ixy="0" ixz="0"
+                iyy="${small_inertial_value}" iyz="0" izz="${small_inertial_value}"/>
+      </inertial-->
+      <inertial>
+        <mass value="0.03"/>
+        <origin rpy="0 0 0" xyz="0 0 0"/>
+        <inertia ixx="7.2964970814e-05" ixy="0.0" ixz="0.0" iyy="7.6464969414e-05" iyz="0.0" izz="6.62499735e-06"/>
       </inertial>
     </link>
@@ -377,9 +441,14 @@
         </geometry>
       </collision>
-      <inertial>
-        <mass value="${small_mass}"/>
-        <origin rpy="0 0 0" xyz="0 0 0"/>
-        <inertia ixx="${small_inertial_value}" ixy="0" ixz="0"
-                iyy="${small_inertial_value}" iyz="0" izz="${small_inertial_value}"/>
+      <!--inertial>
+        <mass value="${small_mass}"/>
+        <origin rpy="0 0 0" xyz="0 0 0"/>
+        <inertia ixx="${small_inertial_value}" ixy="0" ixz="0"
+                iyy="${small_inertial_value}" iyz="0" izz="${small_inertial_value}"/>
+      </inertial-->
+      <inertial>
+        <mass value="0.03"/>
+        <origin rpy="0 0 0" xyz="0 0 0"/>
+        <inertia ixx="7.2964970814e-05" ixy="0.0" ixz="0.0" iyy="7.6464969414e-05" iyz="0.0" izz="6.62499735e-06"/>
       </inertial>
     </link>

Commit message: Changed the parameters values from Grasping Plugin

File: xacro/ist_cyton_gamma_1500_macros.urdf.xacro (robot description, xacro)
@@ -405,5 +405,6 @@
         <origin rpy="0 -0.05 0" xyz="0.014 -0.001 -0.07"/>
         <geometry>
-          <box size="0.045 0.025 0.169"/>
+          <!--box size="0.045 0.025 0.169"/-->
+          <box size="0.04 0.07 0.165"/>
         </geometry>
       </collision>
@@ -438,5 +439,5 @@
         <origin rpy="0 0.1 0" xyz="-0.02 0.024 -0.07"/>
         <geometry>
-          <box size="0.045 0.07 0.165"/>
+          <box size="0.04 0.07 0.165"/>
         </geometry>
       </collision>
@@ -596,7 +597,7 @@
         <forces_angle_tolerance>100</forces_angle_tolerance>
         <update_rate>4</update_rate>
-        <grip_count_threshold>4</grip_count_threshold>
+        <grip_count_threshold>1</grip_count_threshold>
         <max_grip_count>8</max_grip_count>
-        <release_tolerance>0.005</release_tolerance>
+        <release_tolerance>0.003</release_tolerance>
         <disable_collisions_on_attach>false</disable_collisions_on_attach>
         <contact_topic>__default_topic__</contact_topic>

Commit message: I changed the collision boxes of the fingers and the parameters on the grasping library.

File: xacro/ist_cyton_gamma_1500_macros.urdf.xacro (robot description, xacro)
@@ -403,5 +403,5 @@
       </visual>
       <collision>
-        <origin rpy="0 -0.05 0" xyz="0.014 -0.001 -0.07"/>
+        <origin rpy="0 0 0" xyz="0.014 -0.001 -0.07"/>
         <geometry>
           <!--box size="0.045 0.025 0.169"/-->
@@ -437,5 +437,5 @@
       </visual>
       <collision>
-        <origin rpy="0 0.1 0" xyz="-0.02 0.024 -0.07"/>
+        <origin rpy="0 0 0" xyz="-0.02 0.024 -0.07"/>
         <geometry>
           <box size="0.04 0.07 0.165"/>
@@ -596,8 +596,8 @@
         </arm>
         <forces_angle_tolerance>100</forces_angle_tolerance>
-        <update_rate>4</update_rate>
+        <update_rate>0.5</update_rate>
         <grip_count_threshold>1</grip_count_threshold>
         <max_grip_count>8</max_grip_count>
-        <release_tolerance>0.003</release_tolerance>
+        <release_tolerance>0.005</release_tolerance>
         <disable_collisions_on_attach>false</disable_collisions_on_attach>
         <contact_topic>__default_topic__</contact_topic>

Commit message: [last commit from lisbon] add checkerboard to arm urdf

File: xacro/ist_cyton_gamma_1500_macros.urdf.xacro (robot description, xacro)
@@ -403,5 +403,5 @@
       </visual>
       <collision>
-        <origin rpy="0 0 0" xyz="0.014 -0.001 -0.07"/>
+        <origin rpy="0 -0.05 0" xyz="0.014 -0.001 -0.07"/>
         <geometry>
           <!--box size="0.045 0.025 0.169"/-->
@@ -437,5 +437,5 @@
       </visual>
       <collision>
-        <origin rpy="0 0 0" xyz="-0.02 0.024 -0.07"/>
+        <origin rpy="0 0.1 0" xyz="-0.02 0.024 -0.07"/>
         <geometry>
           <box size="0.04 0.07 0.165"/>
@@ -472,4 +472,31 @@
       <mimic joint="${prefix}gripper_joint" multiplier="-1" offset="0"/>
     </joint>
+    <link name="${prefix}virtual_checkerboard">
+      <visual>
+        <origin xyz="0 0 0" rpy="0 0 0" />
+        <geometry>
+          <sphere radius="0.002" />
+        </geometry>
+        <material name="grey">
+          <color rgba="0.7 0.7 0.7 0.8" />
+        </material>
+      </visual>
+    </link>
+    <joint name="${prefix}virtual_checkerboard_joint" type="fixed">
+      <parent link="${prefix}Motor_+_Base" />
+      <child link="${prefix}virtual_checkerboard" />
+      <origin xyz="0.0 0.03 0.0" rpy="0 ${M_PI/2} 0" />
+    </joint>
+    <link name="${prefix}virtual_endeffector">
+      <visual>
+        <origin xyz="0 0 0" rpy="0 0 0" />
+        <geometry>
+          <sphere radius="0.002" />
+        </geometry>
+        <material name="grey">
+          <color rgba="0.7 0.7 0.7 0.8" />
+        </material>
+      </visual>
+    </link>
     <joint name="${prefix}virtual_endeffector_joint" type="fixed">
       <parent link="${prefix}Wrist" />
@@ -477,15 +504,4 @@
       <origin xyz="-0.012 0.018 -0.130" rpy="0 0 0" /> <!-- set this value also in mbot pregrasp planning gripper matrix -->
     </joint>
-    <link name="${prefix}virtual_endeffector">
-      <visual>
-        <origin xyz="0 0 0" rpy="0 0 0" />
-        <geometry>
-          <sphere radius="0.002" />
-        </geometry>
-        <material name="grey">
-          <color rgba="0.7 0.7 0.7 0.8" />
-        </material>
-      </visual>
-    </link>
     <!-- Camera -->
     <!-- Camera: Colour : Base_Camera_link -->
@@ -596,8 +612,8 @@
         </arm>
         <forces_angle_tolerance>100</forces_angle_tolerance>
-        <update_rate>0.5</update_rate>
+        <update_rate>4</update_rate>
         <grip_count_threshold>1</grip_count_threshold>
         <max_grip_count>8</max_grip_count>
-        <release_tolerance>0.005</release_tolerance>
+        <release_tolerance>0.003</release_tolerance>
         <disable_collisions_on_attach>false</disable_collisions_on_attach>
         <contact_topic>__default_topic__</contact_topic>

Commit message: Interim changes to tec gripper, made during RoboCup

File: xacro/ist_cyton_gamma_1500_macros.urdf.xacro (robot description, xacro)
@@ -336,5 +336,5 @@
       <parent link="${prefix}Motor_+_Base" />
       <child link="${prefix}right_link_back" />
-      <origin xyz="0.025 -0.0085 0.015" rpy="0 ${gripper_angular_offset} 0" />
+      <origin xyz="0.025 -0.05 0.015" rpy="0 ${gripper_angular_offset} 0" />
       <axis xyz="0 1 0" />
       <limit effort="1000.0" lower="${gripper_lower_limit}" upper="${gripper_upper_limit}" velocity="0.5"/>
@@ -343,5 +343,5 @@
     <link name="${prefix}left_link_front">
       <visual>
-        <origin rpy="0 3.142 0" xyz="0 0 0"/>
+        <origin rpy="0 2.842 0" xyz="0 0 0"/>
         <geometry>
           <mesh filename="package://cyton_gamma_1500_description/meshes/gripper/left_front_link.dae"/>
@@ -363,5 +363,5 @@
       <parent link="${prefix}Motor_+_Base" />
       <child link="${prefix}left_link_front" />
-      <origin xyz="-0.022 -0.001 0" rpy="0 -${gripper_angular_offset} 0" />
+      <origin xyz="-0.024 -0.001 0.021" rpy="0 -${gripper_angular_offset} 0" />
       <axis xyz="0 1 0" />
       <limit effort="1000.0" lower="${-gripper_upper_limit}" upper="${-gripper_lower_limit}" velocity="0.5"/>
@@ -390,5 +390,5 @@
       <parent link="${prefix}Motor_+_Base" />
       <child link="${prefix}left_link_back" />
-      <origin xyz="-0.0469 -0.014 0.0155" rpy="0 -${gripper_angular_offset} 0" />
+      <origin xyz="-0.049 -0.017 0.0308" rpy="0 -${gripper_angular_offset} 0" />
       <axis xyz="0 1 0" />
       <limit effort="1000.0" lower="${-gripper_upper_limit}" upper="${-gripper_lower_limit}" velocity="0.5"/>
@@ -424,5 +424,5 @@
       <parent link="${prefix}left_link_back" />
       <child link="${prefix}one_finger" />
-      <origin xyz="-0.06 0.008 0.0" rpy="0 ${gripper_angular_offset} 0" />
+      <origin xyz="-0.06 -0.001 0.0" rpy="0 ${gripper_angular_offset} 0" />
       <axis xyz="0 1 0" />
       <limit effort="1000.0" lower="${gripper_lower_limit}" upper="${gripper_upper_limit}" velocity="0.5"/>
